Commit message: Modify the package

File: panda_description/urdf/hand.urdf.xacro (robot description, xacro)
@@ -2,4 +2,4 @@
 <robot xmlns:xacro="http://www.ros.org/wiki/xacro" name="hand">
   <xacro:include filename="$(find panda_description)/urdf/hand.xacro" />
-  <xacro:hand ns="panda"/>
+  <xacro:hand ns="panda" />
 </robot>

File: panda_description/urdf/hand.xacro (robot description, xacro)
@@ -4,7 +4,7 @@
     <xacro:unless value="${connected_to == ''}">
       <joint name="${ns}_hand_joint" type="fixed">
-        <parent link="${connected_to}"/>
-        <child link="${ns}_hand"/>
-        <origin xyz="${xyz}" rpy="${rpy}"/>
+        <parent link="${connected_to}" />
+        <child link="${ns}_hand" />
+        <origin xyz="${xyz}" rpy="${rpy}" />
       </joint>
     </xacro:unless>
@@ -12,10 +12,10 @@
       <visual>
         <geometry>
-          <mesh filename="package://panda_description/meshes/visual/hand.dae"/>
+          <mesh filename="package://panda_description/meshes/visual/hand.dae" />
         </geometry>
       </visual>
       <collision>
         <geometry>
-          <mesh filename="package://panda_description/meshes/collision/hand.stl"/>
+          <mesh filename="package://panda_description/meshes/collision/hand.stl" />
         </geometry>
       </collision>
@@ -24,10 +24,10 @@
       <visual>
         <geometry>
-          <mesh filename="package://panda_description/meshes/visual/finger.dae"/>
+          <mesh filename="package://panda_description/meshes/visual/finger.dae" />
         </geometry>
       </visual>
       <collision>
         <geometry>
-          <mesh filename="package://panda_description/meshes/collision/finger.stl"/>
+          <mesh filename="package://panda_description/meshes/collision/finger.stl" />
         </geometry>
       </collision>
@@ -35,29 +35,29 @@
     <link name="${ns}_rightfinger">
       <visual>
-        <origin xyz="0 0 0" rpy="0 0 ${pi}"/>
+        <origin xyz="0 0 0" rpy="0 0 ${pi}" />
         <geometry>
-          <mesh filename="package://panda_description/meshes/visual/finger.dae"/>
+          <mesh filename="package://panda_description/meshes/visual/finger.dae" />
         </geometry>
       </visual>
       <collision>
-        <origin xyz="0 0 0" rpy="0 0 ${pi}"/>
+        <origin xyz="0 0 0" rpy="0 0 ${pi}" />
         <geometry>
-          <mesh filename="package://panda_description/meshes/collision/finger.stl"/>
+          <mesh filename="package://panda_description/meshes/collision/finger.stl" />
         </geometry>
       </collision>
     </link>
     <joint name="${ns}_finger_joint1" type="prismatic">
-      <parent link="${ns}_hand"/>
-      <child link="${ns}_leftfinger"/>
-      <origin xyz="0 0 0.0584" rpy="0 0 0"/>
-      <axis xyz="0 1 0"/>
-      <limit effort="20" lower="0.0" upper="0.04" velocity="0.2"/>
+      <parent link="${ns}_hand" />
+      <child link="${ns}_leftfinger" />
+      <origin xyz="0 0 0.0584" rpy="0 0 0" />
+      <axis xyz="0 1 0" />
+      <limit effort="20" lower="0.0" upper="0.04" velocity="0.2" />
     </joint>
     <joint name="${ns}_finger_joint2" type="prismatic">
-      <parent link="${ns}_hand"/>
-      <child link="${ns}_rightfinger"/>
-      <origin xyz="0 0 0.0584" rpy="0 0 0"/>
-      <axis xyz="0 -1 0"/>
-      <limit effort="20" lower="0.0" upper="0.04" velocity="0.2"/>
+      <parent link="${ns}_hand" />
+      <child link="${ns}_rightfinger" />
+      <origin xyz="0 0 0.0584" rpy="0 0 0" />
+      <axis xyz="0 -1 0" />
+      <limit effort="20" lower="0.0" upper="0.04" velocity="0.2" />
       <mimic joint="${ns}_finger_joint1" />
     </joint>

File: panda_description/urdf/panda_arm.xacro (robot description, xacro)
@@ -4,7 +4,7 @@
     <xacro:unless value="${not connected_to}">
       <joint name="${arm_id}_joint_${connected_to}" type="fixed">
-        <parent link="${connected_to}"/>
-        <child link="${arm_id}_link0"/>
-        <origin rpy="${rpy}" xyz="${xyz}"/>
+        <parent link="${connected_to}" />
+        <child link="${arm_id}_link0" />
+        <origin rpy="${rpy}" xyz="${xyz}" />
       </joint>
     </xacro:unless>
@@ -12,10 +12,10 @@
       <visual>
         <geometry>
-          <mesh filename="package://${description_pkg}/meshes/visual/link0.dae"/>
+          <mesh filename="package://${description_pkg}/meshes/visual/link0.dae" />
         </geometry>
       </visual>
       <collision>
         <geometry>
-          <mesh filename="package://${description_pkg}/meshes/collision/link0.stl"/>
+          <mesh filename="package://${description_pkg}/meshes/collision/link0.stl" />
         </geometry>
       </collision>
@@ -24,40 +24,40 @@
       <visual>
         <geometry>
-          <mesh filename="package://${description_pkg}/meshes/visual/link1.dae"/>
+          <mesh filename="package://${description_pkg}/meshes/visual/link1.dae" />
         </geometry>
       </visual>
       <collision>
         <geometry>
-          <mesh filename="package://${description_pkg}/meshes/collision/link1.stl"/>
+          <mesh filename="package://${description_pkg}/meshes/collision/link1.stl" />
         </geometry>
       </collision>
     </link>
     <joint name="${arm_id}_joint1" type="revolute">
-      <safety_controller k_position="100.0" k_velocity="40.0" soft_lower_limit="-2.8973" soft_upper_limit="2.8973"/>
-      <origin rpy="0 0 0" xyz="0 0 0.333"/>
-      <parent link="${arm_id}_link0"/>
-      <child link="${arm_id}_link1"/>
-      <axis xyz="0 0 1"/>
-      <limit effort="87" lower="-2.9671" upper="2.9671" velocity="2.3925"/>
+      <safety_controller k_position="100.0" k_velocity="40.0" soft_lower_limit="-2.8973" soft_upper_limit="2.8973" />
+      <origin rpy="0 0 0" xyz="0 0 0.333" />
+      <parent link="${arm_id}_link0" />
+      <child link="${arm_id}_link1" />
+      <axis xyz="0 0 1" />
+      <limit effort="87" lower="-2.9671" upper="2.9671" velocity="2.3925" />
     </joint>
     <link name="${arm_id}_link2">
       <visual>
         <geometry>
-          <mesh filename="package://${description_pkg}/meshes/visual/link2.dae"/>
+          <mesh filename="package://${description_pkg}/meshes/visual/link2.dae" />
         </geometry>
       </visual>
       <collision>
         <geometry>
-          <mesh filename="package://${description_pkg}/meshes/collision/link2.stl"/>
+          <mesh filename="package://${description_pkg}/meshes/collision/link2.stl" />
         </geometry>
       </collision>
     </link>
     <joint name="${arm_id}_joint2" type="revolute">
-      <safety_controller k_position="100.0" k_velocity="40.0" soft_lower_limit="-1.7628" soft_upper_limit="1.7628"/>
-      <origin rpy="${-pi/2} 0 0" xyz="0 0 0"/>
-      <parent link="${arm_id}_link1"/>
-      <child link="${arm_id}_link2"/>
-      <axis xyz="0 0 1"/>
-      <limit effort="87" lower="-1.8326" upper="1.8326" velocity="2.3925"/>
+      <safety_controller k_position="100.0" k_velocity="40.0" soft_lower_limit="-1.7628" soft_upper_limit="1.7628" />
+      <origin rpy="${-pi/2} 0 0" xyz="0 0 0" />
+      <parent link="${arm_id}_link1" />
+      <child link="${arm_id}_link2" />
+      <axis xyz="0 0 1" />
+      <limit effort="87" lower="-1.8326" upper="1.8326" velocity="2.3925" />
     </joint>
     <link name="${arm_id}_link3">
@@ -69,102 +69,102 @@
       <collision>
         <geometry>
-          <mesh filename="package://${description_pkg}/meshes/collision/link3.stl"/>
+          <mesh filename="package://${description_pkg}/meshes/collision/link3.stl" />
         </geometry>
       </collision>
     </link>
     <joint name="${arm_id}_joint3" type="revolute">
-      <safety_controller k_position="100.0" k_velocity="40.0" soft_lower_limit="-2.8973" soft_upper_limit="2.8973"/>
-      <origin rpy="${pi/2} 0 0" xyz="0 -0.316 0"/>
-      <parent link="${arm_id}_link2"/>
-      <child link="${arm_id}_link3"/>
-      <axis xyz="0 0 1"/>
-      <limit effort="87" lower="-2.9671" upper="2.9671" velocity="2.3925"/>
+      <safety_controller k_position="100.0" k_velocity="40.0" soft_lower_limit="-2.8973" soft_upper_limit="2.8973" />
+      <origin rpy="${pi/2} 0 0" xyz="0 -0.316 0" />
+      <parent link="${arm_id}_link2" />
+      <child link="${arm_id}_link3" />
+      <axis xyz="0 0 1" />
+      <limit effort="87" lower="-2.9671" upper="2.9671" velocity="2.3925" />
     </joint>
     <link name="${arm_id}_link4">
       <visual>
         <geometry>
-          <mesh filename="package://${description_pkg}/meshes/visual/link4.dae"/>
+          <mesh filename="package://${description_pkg}/meshes/visual/link4.dae" />
         </geometry>
       </visual>
       <collision>
         <geometry>
-          <mesh filename="package://${description_pkg}/meshes/collision/link4.stl"/>
+          <mesh filename="package://${description_pkg}/meshes/collision/link4.stl" />
         </geometry>
       </collision>
     </link>
     <joint name="${arm_id}_joint4" type="revolute">
-      <safety_controller k_position="100.0" k_velocity="40.0" soft_lower_limit="-3.0718" soft_upper_limit="0.0175"/>
-      <origin rpy="${pi/2} 0 0" xyz="0.0825 0 0"/>
-      <parent link="${arm_id}_link3"/>
-      <child link="${arm_id}_link4"/>
-      <axis xyz="0 0 1"/>
-      <limit effort="87" lower="-3.1416" upper="0.0873" velocity="2.3925"/>
+      <safety_controller k_position="100.0" k_velocity="40.0" soft_lower_limit="-3.0718" soft_upper_limit="0.0175" />
+      <origin rpy="${pi/2} 0 0" xyz="0.0825 0 0" />
+      <parent link="${arm_id}_link3" />
+      <child link="${arm_id}_link4" />
+      <axis xyz="0 0 1" />
+      <limit effort="87" lower="-3.1416" upper="0.0873" velocity="2.3925" />
     </joint>
     <link name="${arm_id}_link5">
       <visual>
         <geometry>
-          <mesh filename="package://${description_pkg}/meshes/visual/link5.dae"/>
+          <mesh filename="package://${description_pkg}/meshes/visual/link5.dae" />
         </geometry>
       </visual>
       <collision>
         <geometry>
-          <mesh filename="package://${description_pkg}/meshes/collision/link5.stl"/>
+          <mesh filename="package://${description_pkg}/meshes/collision/link5.stl" />
         </geometry>
       </collision>
     </link>
     <joint name="${arm_id}_joint5" type="revolute">
-      <safety_controller k_position="100.0" k_velocity="40.0" soft_lower_limit="-2.8973" soft_upper_limit="2.8973"/>
-      <origin rpy="${-pi/2} 0 0" xyz="-0.0825 0.384 0"/>
-      <parent link="${arm_id}_link4"/>
-      <child link="${arm_id}_link5"/>
-      <axis xyz="0 0 1"/>
-      <limit effort="12" lower="-2.9671" upper="2.9671" velocity="2.8710"/>
+      <safety_controller k_position="100.0" k_velocity="40.0" soft_lower_limit="-2.8973" soft_upper_limit="2.8973" />
+      <origin rpy="${-pi/2} 0 0" xyz="-0.0825 0.384 0" />
+      <parent link="${arm_id}_link4" />
+      <child link="${arm_id}_link5" />
+      <axis xyz="0 0 1" />
+      <limit effort="12" lower="-2.9671" upper="2.9671" velocity="2.8710" />
     </joint>
     <link name="${arm_id}_link6">
       <visual>
         <geometry>
-          <mesh filename="package://${description_pkg}/meshes/visual/link6.dae"/>
+          <mesh filename="package://${description_pkg}/meshes/visual/link6.dae" />
         </geometry>
       </visual>
       <collision>
         <geometry>
-          <mesh filename="package://${description_pkg}/meshes/collision/link6.stl"/>
+          <mesh filename="package://${description_pkg}/meshes/collision/link6.stl" />
         </geometry>
       </collision>
     </link>
     <joint name="${arm_id}_joint6" type="revolute">
-      <safety_controller k_position="100.0" k_velocity="40.0" soft_lower_limit="-0.0175" soft_upper_limit="3.7525"/>
-      <origin rpy="${pi/2} 0 0" xyz="0 0 0"/>
-      <parent link="${arm_id}_link5"/>
-      <child link="${arm_id}_link6"/>
-      <axis xyz="0 0 1"/>
-      <limit effort="12" lower="-0.0873" upper="3.8223" velocity="2.8710"/>
+      <safety_controller k_position="100.0" k_velocity="40.0" soft_lower_limit="-0.0175" soft_upper_limit="3.7525" />
+      <origin rpy="${pi/2} 0 0" xyz="0 0 0" />
+      <parent link="${arm_id}_link5" />
+      <child link="${arm_id}_link6" />
+      <axis xyz="0 0 1" />
+      <limit effort="12" lower="-0.0873" upper="3.8223" velocity="2.8710" />
     </joint>
     <link name="${arm_id}_link7">
       <visual>
         <geometry>
-          <mesh filename="package://${description_pkg}/meshes/visual/link7.dae"/>
+          <mesh filename="package://${description_pkg}/meshes/visual/link7.dae" />
         </geometry>
       </visual>
       <collision>
         <geometry>
-          <mesh filename="package://${description_pkg}/meshes/collision/link7.stl"/>
+          <mesh filename="package://${description_pkg}/meshes/collision/link7.stl" />
         </geometry>
       </collision>
     </link>
     <joint name="${arm_id}_joint7" type="revolute">
-      <safety_controller k_position="100.0" k_velocity="40.0" soft_lower_limit="-2.8973" soft_upper_limit="2.8973"/>
-      <origin rpy="${pi/2} 0 0" xyz="0.088 0 0"/>
-      <parent link="${arm_id}_link6"/>
-      <child link="${arm_id}_link7"/>
-      <axis xyz="0 0 1"/>
-      <limit effort="12" lower="-2.9671" upper="2.9671" velocity="2.8710"/>
+      <safety_controller k_position="100.0" k_velocity="40.0" soft_lower_limit="-2.8973" soft_upper_limit="2.8973" />
+      <origin rpy="${pi/2} 0 0" xyz="0.088 0 0" />
+      <parent link="${arm_id}_link6" />
+      <child link="${arm_id}_link7" />
+      <axis xyz="0 0 1" />
+      <limit effort="12" lower="-2.9671" upper="2.9671" velocity="2.8710" />
     </joint>
-    <link name="${arm_id}_link8"/>
+    <link name="${arm_id}_link8" />
     <joint name="${arm_id}_joint8" type="fixed">
-      <origin rpy="0 0 0" xyz="0 0 0.107"/>
-      <parent link="${arm_id}_link7"/>
-      <child link="${arm_id}_link8"/>
-      <axis xyz="0 0 0"/>
+      <origin rpy="0 0 0" xyz="0 0 0.107" />
+      <parent link="${arm_id}_link7" />
+      <child link="${arm_id}_link8" />
+      <axis xyz="0 0 0" />
     </joint>
   </xacro:macro>

File: panda_description/urdf/panda_arm_hand.urdf.xacro (robot description, xacro)
@@ -1,7 +1,7 @@
 <?xml version="1.0" encoding="utf-8"?>
 <robot xmlns:xacro="http://www.ros.org/wiki/xacro" name="panda">
-  <xacro:include filename="$(find panda_description)/urdf/panda_arm.xacro"/>
-  <xacro:include filename="$(find panda_description)/urdf/hand.xacro"/>
+  <xacro:include filename="$(find panda_description)/urdf/panda_arm.xacro" />
+  <xacro:include filename="$(find panda_description)/urdf/hand.xacro" />
   <xacro:panda_arm />
-  <xacro:hand ns="panda" rpy="0 0 ${-pi/4}" connected_to="panda_link8"/>
+  <xacro:hand ns="panda" rpy="0 0 ${-pi/4}" connected_to="panda_link8" />
 </robot>
