Commit message: Modify the file

File: panda_description/urdf/panda_arm.xacro (robot description, xacro)
@@ -38,5 +38,5 @@
       </collision>
       <inertial>
-        <origin xyz="0 0 0.0125" rpy="0 0 0" />
+        <origin xyz="0 0 -0.08" rpy="0 0 0" />
         <mass value="1" />
         <inertia ixx="1" ixy="0" ixz="0" iyy="1" iyz="0" izz="1" />
@@ -63,7 +63,9 @@
       </collision>
       <inertial>
-        <origin xyz="0 0 0.5" rpy="0 0 0" />
-        <mass value="1" />
-        <inertia ixx="1" ixy="0" ixz="0" iyy="1" iyz="0" izz="1" />
+        <origin xyz="0 -0.05 0" rpy="0 0 0" />
+        <mass value="1" />
+        <inertia ixx="-1" ixy="0" ixz="0"
+                 iyy="-1" iyz="0"
+                 izz="-1" />
       </inertial>
     </link>
@@ -88,5 +90,5 @@
       </collision>
 <!--       <inertial>
-        <origin xyz="0 0 0.5" rpy="0 0 0" />
+        <origin xyz="0 0 0" rpy="0 0 0" />
         <mass value="1" />
         <inertia ixx="1" ixy="0" ixz="0" iyy="1" iyz="0" izz="1" />
