Commit message: Modify inertial tag

File: panda_description/urdf/hand.xacro (robot description, xacro)
@@ -20,4 +20,9 @@
         </geometry>
       </collision>
+<!--       <inertial>
+        <origin xyz="0 0 0.25" rpy="0 0 0" />
+        <mass value="0.5" />
+        <inertia ixx="1" ixy="0" ixz="0" iyy="1" iyz="0" izz="1" />
+      </inertial> -->
     </link>
     <link name="${ns}_leftfinger">
@@ -32,4 +37,9 @@
         </geometry>
       </collision>
+<!--       <inertial>
+        <origin xyz="0 0 0.25" rpy="0 0 0" />
+        <mass value="0.25" />
+        <inertia ixx="1" ixy="0" ixz="0" iyy="1" iyz="0" izz="1" />
+      </inertial> -->
     </link>
     <link name="${ns}_rightfinger">
@@ -46,4 +56,9 @@
         </geometry>
       </collision>
+<!--       <inertial>
+        <origin xyz="0 0 0.25" rpy="0 0 0" />
+        <mass value="0.25" />
+        <inertia ixx="1" ixy="0" ixz="0" iyy="1" iyz="0" izz="1" />
+      </inertial> -->
     </link>
     <joint name="${ns}_finger_joint1" type="prismatic">

File: panda_description/urdf/panda_arm.xacro (robot description, xacro)
@@ -21,7 +21,7 @@
       </collision>
       <inertial>
-        <origin xyz="0 0 0" rpy="0 0 0" />
-        <mass value="1" />
-        <inertia ixx="0" ixy="0" ixz="0" iyy="0" iyz="0" izz="0" />
+        <origin xyz="0 0 0.05" rpy="0 0 0" />
+        <mass value="1" />
+        <inertia ixx="1" ixy="0" ixz="0" iyy="1" iyz="0" izz="1" />
       </inertial>
     </link>
@@ -38,7 +38,7 @@
       </collision>
       <inertial>
-        <origin xyz="0 0 0" rpy="0 0 0" />
-        <mass value="1" />
-        <inertia ixx="0" ixy="0" ixz="0" iyy="0" iyz="0" izz="0" />
+        <origin xyz="0 0 0.0125" rpy="0 0 0" />
+        <mass value="1" />
+        <inertia ixx="1" ixy="0" ixz="0" iyy="1" iyz="0" izz="1" />
       </inertial>
     </link>
@@ -63,7 +63,7 @@
       </collision>
       <inertial>
-        <origin xyz="0 0 0" rpy="0 0 0" />
-        <mass value="1" />
-        <inertia ixx="0" ixy="0" ixz="0" iyy="0" iyz="0" izz="0" />
+        <origin xyz="0 0 0.5" rpy="0 0 0" />
+        <mass value="1" />
+        <inertia ixx="1" ixy="0" ixz="0" iyy="1" iyz="0" izz="1" />
       </inertial>
     </link>
@@ -87,9 +87,9 @@
         </geometry>
       </collision>
-      <inertial>
-        <origin xyz="0 0 0" rpy="0 0 0" />
-        <mass value="1" />
-        <inertia ixx="0" ixy="0" ixz="0" iyy="0" iyz="0" izz="0" />
-      </inertial>
+<!--       <inertial>
+        <origin xyz="0 0 0.5" rpy="0 0 0" />
+        <mass value="1" />
+        <inertia ixx="1" ixy="0" ixz="0" iyy="1" iyz="0" izz="1" />
+      </inertial> -->
     </link>
     <joint name="${arm_id}_joint3" type="revolute">
@@ -112,9 +112,9 @@
         </geometry>
       </collision>
-      <inertial>
-        <origin xyz="0 0 0" rpy="0 0 0" />
-        <mass value="1" />
-        <inertia ixx="0" ixy="0" ixz="0" iyy="0" iyz="0" izz="0" />
-      </inertial>
+<!--       <inertial>
+        <origin xyz="0 0 0.5" rpy="0 0 0" />
+        <mass value="1" />
+        <inertia ixx="1" ixy="0" ixz="0" iyy="1" iyz="0" izz="1" />
+      </inertial> -->
     </link>
     <joint name="${arm_id}_joint4" type="revolute">
@@ -137,9 +137,9 @@
         </geometry>
       </collision>
-      <inertial>
-        <origin xyz="0 0 0" rpy="0 0 0" />
-        <mass value="1" />
-        <inertia ixx="0" ixy="0" ixz="0" iyy="0" iyz="0" izz="0" />
-      </inertial>
+<!--       <inertial>
+        <origin xyz="0 0 0.5" rpy="0 0 0" />
+        <mass value="1" />
+        <inertia ixx="1" ixy="0" ixz="0" iyy="1" iyz="0" izz="1" />
+      </inertial> -->
     </link>
     <joint name="${arm_id}_joint5" type="revolute">
@@ -162,9 +162,9 @@
         </geometry>
       </collision>
-      <inertial>
-        <origin xyz="0 0 0" rpy="0 0 0" />
-        <mass value="1" />
-        <inertia ixx="0" ixy="0" ixz="0" iyy="0" iyz="0" izz="0" />
-      </inertial>
+<!--       <inertial>
+        <origin xyz="0 0 0.5" rpy="0 0 0" />
+        <mass value="1" />
+        <inertia ixx="1" ixy="0" ixz="0" iyy="1" iyz="0" izz="1" />
+      </inertial> -->
     </link>
     <joint name="${arm_id}_joint6" type="revolute">
@@ -187,9 +187,9 @@
         </geometry>
       </collision>
-      <inertial>
-        <origin xyz="0 0 0" rpy="0 0 0" />
-        <mass value="1" />
-        <inertia ixx="0" ixy="0" ixz="0" iyy="0" iyz="0" izz="0" />
-      </inertial>
+<!--       <inertial>
+        <origin xyz="0 0 0.5" rpy="0 0 0" />
+        <mass value="1" />
+        <inertia ixx="1" ixy="0" ixz="0" iyy="1" iyz="0" izz="1" />
+      </inertial> -->
     </link>
     <joint name="${arm_id}_joint7" type="revolute">

Commit message: Modify panda_description package

File: panda_description/urdf/hand.xacro (robot description, xacro)
@@ -23,8 +23,8 @@
         <origin xyz="-2.7600000000e-06 -6.1551000000e-04 2.3929520000e-02"
                 rpy="0 0 0" />
-        <mass value="2.36" />
-        <inertia ixx="8.0087281861e-03"  ixy="-1.3983247099e-06"
-                 ixz="3.1668653650e-07"  iyy="1.6099853693e-03"
-                 iyz="-1.4527159720e-04" izz="7.2469819837e-03" />
+        <mass value="1.0" />
+        <inertia ixx="3.3935288924e-03"  ixy="-5.9251047030e-07"
+                 ixz="1.3418921038e-07"  iyy="6.8219719040e-04"
+                 iyz="-6.1555761524e-05" izz="3.0707550778e-03" />
       </inertial>
     </link>
