Commit message: Modify the files

File: panda_description/gazebo/panda_arm_hand_transmission.xacro (robot description, xacro)
@@ -4,8 +4,8 @@
     <type>transmission_interface/SimpleTransmission</type>
     <joint name="panda_joint1">
-      <hardwareInterface>PositionJointInterface</hardwareInterface>
+      <hardwareInterface>hardware_interface/EffortJointInterface</hardwareInterface>
     </joint>
     <actuator name="joint1_actuator">
-      <hardwareInterface>PositionJointInterface</hardwareInterface>
+      <hardwareInterface>hardware_interface/EffortJointInterface</hardwareInterface>
       <mechanicalReduction>1</mechanicalReduction>
     </actuator>
@@ -14,8 +14,8 @@
     <type>transmission_interface/SimpleTransmission</type>
     <joint name="panda_joint2">
-      <hardwareInterface>PositionJointInterface</hardwareInterface>
+      <hardwareInterface>hardware_interface/EffortJointInterface</hardwareInterface>
     </joint>
     <actuator name="joint2_actuator">
-      <hardwareInterface>PositionJointInterface</hardwareInterface>
+      <hardwareInterface>hardware_interface/EffortJointInterface</hardwareInterface>
       <mechanicalReduction>1</mechanicalReduction>
     </actuator>
@@ -24,8 +24,8 @@
     <type>transmission_interface/SimpleTransmission</type>
     <joint name="panda_joint3">
-      <hardwareInterface>PositionJointInterface</hardwareInterface>
+      <hardwareInterface>hardware_interface/EffortJointInterface</hardwareInterface>
     </joint>
     <actuator name="joint3_actuator">
-      <hardwareInterface>PositionJointInterface</hardwareInterface>
+      <hardwareInterface>hardware_interface/EffortJointInterface</hardwareInterface>
       <mechanicalReduction>1</mechanicalReduction>
     </actuator>
@@ -34,8 +34,8 @@
     <type>transmission_interface/SimpleTransmission</type>
     <joint name="panda_joint4">
-      <hardwareInterface>PositionJointInterface</hardwareInterface>
+      <hardwareInterface>hardware_interface/EffortJointInterface</hardwareInterface>
     </joint>
     <actuator name="joint4_actuator">
-      <hardwareInterface>PositionJointInterface</hardwareInterface>
+      <hardwareInterface>hardware_interface/EffortJointInterface</hardwareInterface>
       <mechanicalReduction>1</mechanicalReduction>
     </actuator>
@@ -44,8 +44,8 @@
     <type>transmission_interface/SimpleTransmission</type>
     <joint name="panda_joint5">
-      <hardwareInterface>PositionJointInterface</hardwareInterface>
+      <hardwareInterface>hardware_interface/EffortJointInterface</hardwareInterface>
     </joint>
     <actuator name="joint5_actuator">
-      <hardwareInterface>PositionJointInterface</hardwareInterface>
+      <hardwareInterface>hardware_interface/EffortJointInterface</hardwareInterface>
       <mechanicalReduction>1</mechanicalReduction>
     </actuator>
@@ -54,8 +54,8 @@
     <type>transmission_interface/SimpleTransmission</type>
     <joint name="panda_joint6">
-      <hardwareInterface>PositionJointInterface</hardwareInterface>
+      <hardwareInterface>hardware_interface/EffortJointInterface</hardwareInterface>
     </joint>
     <actuator name="joint6_actuator">
-      <hardwareInterface>PositionJointInterface</hardwareInterface>
+      <hardwareInterface>hardware_interface/EffortJointInterface</hardwareInterface>
       <mechanicalReduction>1</mechanicalReduction>
     </actuator>
@@ -64,8 +64,28 @@
     <type>transmission_interface/SimpleTransmission</type>
     <joint name="panda_joint7">
-      <hardwareInterface>PositionJointInterface</hardwareInterface>
+      <hardwareInterface>hardware_interface/EffortJointInterface</hardwareInterface>
     </joint>
     <actuator name="joint7_actuator">
-      <hardwareInterface>PositionJointInterface</hardwareInterface>
+      <hardwareInterface>hardware_interface/EffortJointInterface</hardwareInterface>
+      <mechanicalReduction>1</mechanicalReduction>
+    </actuator>
+  </transmission>
+  <transmission name="joint8_simp_trans">
+    <type>transmission_interface/SimpleTransmission</type>
+    <joint name="panda_joint8">
+      <hardwareInterface>hardware_interface/EffortJointInterface</hardwareInterface>
+    </joint>
+    <actuator name="joint8_actuator">
+      <hardwareInterface>hardware_interface/EffortJointInterface</hardwareInterface>
+      <mechanicalReduction>1</mechanicalReduction>
+    </actuator>
+  </transmission>
+  <transmission name="hand_joint_simp_trans">
+    <type>transmission_interface/SimpleTransmission</type>
+    <joint name="panda_hand_joint">
+      <hardwareInterface>hardware_interface/EffortJointInterface</hardwareInterface>
+    </joint>
+    <actuator name="hand_joint_actuator">
+      <hardwareInterface>hardware_interface/EffortJointInterface</hardwareInterface>
       <mechanicalReduction>1</mechanicalReduction>
     </actuator>
@@ -74,8 +94,8 @@
     <type>transmission_interface/SimpleTransmission</type>
     <joint name="panda_finger_joint1">
-      <hardwareInterface>PositionJointInterface</hardwareInterface>
+      <hardwareInterface>hardware_interface/EffortJointInterface</hardwareInterface>
     </joint>
     <actuator name="finger_joint1_actuator">
-      <hardwareInterface>PositionJointInterface</hardwareInterface>
+      <hardwareInterface>hardware_interface/EffortJointInterface</hardwareInterface>
       <mechanicalReduction>1</mechanicalReduction>
     </actuator>
@@ -84,8 +104,8 @@
     <type>transmission_interface/SimpleTransmission</type>
     <joint name="panda_finger_joint2">
-      <hardwareInterface>PositionJointInterface</hardwareInterface>
+      <hardwareInterface>hardware_interface/EffortJointInterface</hardwareInterface>
     </joint>
     <actuator name="finger_joint2_actuator">
-      <hardwareInterface>PositionJointInterface</hardwareInterface>
+      <hardwareInterface>hardware_interface/EffortJointInterface</hardwareInterface>
       <mechanicalReduction>1</mechanicalReduction>
     </actuator>

File: panda_description/gazebo/panda_arm_hand_urdf.xacro (robot description, xacro)
@@ -1,5 +1,63 @@
 <?xml version="1.0" encoding="utf-8"?>
 <robot xmlns:xacro="http://www.ros.org/wiki/xacro">
-<xacro:property name="M_PI" value="3.1415926535897931" />
+<!-- <xacro:property name="M_PI" value="3.1415926535897931" /> -->
+<gazebo reference="panda_link0">
+  <material>Gazebo/Black</material>
+</gazebo>
+<gazebo reference="panda_link1">
+  <mu1>0.2</mu1>
+  <mu2>0.2</mu2>
+  <material>Gazebo/Orange</material>
+</gazebo>
+<gazebo reference="panda_link2">
+  <mu1>0.2</mu1>
+  <mu2>0.2</mu2>
+  <material>Gazebo/Orange</material>
+</gazebo>
+<gazebo reference="panda_link3">
+  <mu1>0.2</mu1>
+  <mu2>0.2</mu2>
+  <material>Gazebo/Orange</material>
+</gazebo>
+<gazebo reference="panda_link4">
+  <mu1>0.2</mu1>
+  <mu2>0.2</mu2>
+  <material>Gazebo/Orange</material>
+</gazebo>
+<gazebo reference="panda_link5">
+  <mu1>0.2</mu1>
+  <mu2>0.2</mu2>
+  <material>Gazebo/Orange</material>
+</gazebo>
+<gazebo reference="panda_link6">
+  <mu1>0.2</mu1>
+  <mu2>0.2</mu2>
+  <material>Gazebo/Orange</material>
+</gazebo>
+<gazebo reference="panda_link7">
+  <mu1>0.2</mu1>
+  <mu2>0.2</mu2>
+  <material>Gazebo/Orange</material>
+</gazebo>
+<gazebo reference="panda_link8">
+  <mu1>0.2</mu1>
+  <mu2>0.2</mu2>
+  <material>Gazebo/Orange</material>
+</gazebo>
+<gazebo reference="panda_hand">
+  <mu1>0.2</mu1>
+  <mu2>0.2</mu2>
+  <material>Gazebo/Orange</material>
+</gazebo>
+<gazebo reference="panda_leftfinger">
+  <mu1>0.2</mu1>
+  <mu2>0.2</mu2>
+  <material>Gazebo/Red</material>
+</gazebo>
+<gazebo reference="panda_rightfinger">
+  <mu1>0.2</mu1>
+  <mu2>0.2</mu2>
+  <material>Gazebo/Red</material>
+</gazebo>
 <!--   <gazebo reference="base_link">
     <kp>10000.0</kp>
@@ -96,5 +154,5 @@
     <material>Gazebo/Grey</material>
   </gazebo> -->
-  <gazebo reference="panda_hand">
+<!--   <gazebo reference="panda_hand">
     <sensor type="depth" name="kinect">
       <update_rate>20</update_rate>
@@ -135,4 +193,4 @@
       </plugin>
     </sensor>
-  </gazebo>
+  </gazebo> -->
 </robot>

File: panda_description/urdf/panda_arm_hand.xacro (robot description, xacro)
@@ -1,4 +1,4 @@
 <?xml version="1.0" encoding="utf-8"?>
-<robot xmlns:xacro="http://www.ros.org/wiki/xacro" name="panda">
+<robot name="panda" xmlns:xacro="http://www.ros.org/wiki/xacro" >
   <xacro:include filename="$(find panda_description)/urdf/panda_arm_hand.urdf.xacro" />
   <xacro:include filename="$(find panda_description)/gazebo/panda_arm_hand.gazebo.xacro" />

Commit message: Delete fixed transmission

File: panda_description/gazebo/panda_arm_hand_transmission.xacro (robot description, xacro)
@@ -4,8 +4,8 @@
     <type>transmission_interface/SimpleTransmission</type>
     <joint name="panda_joint1">
-      <hardwareInterface>hardware_interface/EffortJointInterface</hardwareInterface>
+      <hardwareInterface>hardware_interface/PositionJointInterface</hardwareInterface>
     </joint>
     <actuator name="joint1_actuator">
-      <hardwareInterface>hardware_interface/EffortJointInterface</hardwareInterface>
+      <hardwareInterface>hardware_interface/PositionJointInterface</hardwareInterface>
       <mechanicalReduction>1</mechanicalReduction>
     </actuator>
@@ -14,8 +14,8 @@
     <type>transmission_interface/SimpleTransmission</type>
     <joint name="panda_joint2">
-      <hardwareInterface>hardware_interface/EffortJointInterface</hardwareInterface>
+      <hardwareInterface>hardware_interface/PositionJointInterface</hardwareInterface>
     </joint>
     <actuator name="joint2_actuator">
-      <hardwareInterface>hardware_interface/EffortJointInterface</hardwareInterface>
+      <hardwareInterface>hardware_interface/PositionJointInterface</hardwareInterface>
       <mechanicalReduction>1</mechanicalReduction>
     </actuator>
@@ -24,8 +24,8 @@
     <type>transmission_interface/SimpleTransmission</type>
     <joint name="panda_joint3">
-      <hardwareInterface>hardware_interface/EffortJointInterface</hardwareInterface>
+      <hardwareInterface>hardware_interface/PositionJointInterface</hardwareInterface>
     </joint>
     <actuator name="joint3_actuator">
-      <hardwareInterface>hardware_interface/EffortJointInterface</hardwareInterface>
+      <hardwareInterface>hardware_interface/PositionJointInterface</hardwareInterface>
       <mechanicalReduction>1</mechanicalReduction>
     </actuator>
@@ -34,8 +34,8 @@
     <type>transmission_interface/SimpleTransmission</type>
     <joint name="panda_joint4">
-      <hardwareInterface>hardware_interface/EffortJointInterface</hardwareInterface>
+      <hardwareInterface>hardware_interface/PositionJointInterface</hardwareInterface>
     </joint>
     <actuator name="joint4_actuator">
-      <hardwareInterface>hardware_interface/EffortJointInterface</hardwareInterface>
+      <hardwareInterface>hardware_interface/PositionJointInterface</hardwareInterface>
       <mechanicalReduction>1</mechanicalReduction>
     </actuator>
@@ -44,8 +44,8 @@
     <type>transmission_interface/SimpleTransmission</type>
     <joint name="panda_joint5">
-      <hardwareInterface>hardware_interface/EffortJointInterface</hardwareInterface>
+      <hardwareInterface>hardware_interface/PositionJointInterface</hardwareInterface>
     </joint>
     <actuator name="joint5_actuator">
-      <hardwareInterface>hardware_interface/EffortJointInterface</hardwareInterface>
+      <hardwareInterface>hardware_interface/PositionJointInterface</hardwareInterface>
       <mechanicalReduction>1</mechanicalReduction>
     </actuator>
@@ -54,8 +54,8 @@
     <type>transmission_interface/SimpleTransmission</type>
     <joint name="panda_joint6">
-      <hardwareInterface>hardware_interface/EffortJointInterface</hardwareInterface>
+      <hardwareInterface>hardware_interface/PositionJointInterface</hardwareInterface>
     </joint>
     <actuator name="joint6_actuator">
-      <hardwareInterface>hardware_interface/EffortJointInterface</hardwareInterface>
+      <hardwareInterface>hardware_interface/PositionJointInterface</hardwareInterface>
       <mechanicalReduction>1</mechanicalReduction>
     </actuator>
@@ -64,28 +64,8 @@
     <type>transmission_interface/SimpleTransmission</type>
     <joint name="panda_joint7">
-      <hardwareInterface>hardware_interface/EffortJointInterface</hardwareInterface>
+      <hardwareInterface>hardware_interface/PositionJointInterface</hardwareInterface>
     </joint>
     <actuator name="joint7_actuator">
-      <hardwareInterface>hardware_interface/EffortJointInterface</hardwareInterface>
-      <mechanicalReduction>1</mechanicalReduction>
-    </actuator>
-  </transmission>
-  <transmission name="joint8_simp_trans">
-    <type>transmission_interface/SimpleTransmission</type>
-    <joint name="panda_joint8">
-      <hardwareInterface>hardware_interface/EffortJointInterface</hardwareInterface>
-    </joint>
-    <actuator name="joint8_actuator">
-      <hardwareInterface>hardware_interface/EffortJointInterface</hardwareInterface>
-      <mechanicalReduction>1</mechanicalReduction>
-    </actuator>
-  </transmission>
-  <transmission name="hand_joint_simp_trans">
-    <type>transmission_interface/SimpleTransmission</type>
-    <joint name="panda_hand_joint">
-      <hardwareInterface>hardware_interface/EffortJointInterface</hardwareInterface>
-    </joint>
-    <actuator name="hand_joint_actuator">
-      <hardwareInterface>hardware_interface/EffortJointInterface</hardwareInterface>
+      <hardwareInterface>hardware_interface/PositionJointInterface</hardwareInterface>
       <mechanicalReduction>1</mechanicalReduction>
     </actuator>
@@ -94,8 +74,8 @@
     <type>transmission_interface/SimpleTransmission</type>
     <joint name="panda_finger_joint1">
-      <hardwareInterface>hardware_interface/EffortJointInterface</hardwareInterface>
+      <hardwareInterface>hardware_interface/PositionJointInterface</hardwareInterface>
     </joint>
     <actuator name="finger_joint1_actuator">
-      <hardwareInterface>hardware_interface/EffortJointInterface</hardwareInterface>
+      <hardwareInterface>hardware_interface/PositionJointInterface</hardwareInterface>
       <mechanicalReduction>1</mechanicalReduction>
     </actuator>
@@ -104,8 +84,8 @@
     <type>transmission_interface/SimpleTransmission</type>
     <joint name="panda_finger_joint2">
-      <hardwareInterface>hardware_interface/EffortJointInterface</hardwareInterface>
+      <hardwareInterface>hardware_interface/PositionJointInterface</hardwareInterface>
     </joint>
     <actuator name="finger_joint2_actuator">
-      <hardwareInterface>hardware_interface/EffortJointInterface</hardwareInterface>
+      <hardwareInterface>hardware_interface/PositionJointInterface</hardwareInterface>
       <mechanicalReduction>1</mechanicalReduction>
     </actuator>
