Commit message: Modify inertial tag

File: panda_description/gazebo/panda_arm_hand_ros_control.xacro (robot description, xacro)
@@ -3,5 +3,5 @@
   <gazebo>
     <plugin name="gazebo_ros_control" filename="libgazebo_ros_control.so">
-    <robotNamespace>/panda</robotNamespace>
+    <robotNamespace>/</robotNamespace>
     <robotSimType>gazebo_ros_control/DefaultRobotHWSim</robotSimType>
     </plugin>

File: panda_description/gazebo/panda_arm_hand_urdf.xacro (robot description, xacro)
@@ -1,7 +1,4 @@
 <?xml version="1.0" encoding="utf-8"?>
 <robot xmlns:xacro="http://www.ros.org/wiki/xacro">
-<!-- <xacro:property name="M_PI" value="3.1415926535897931" /> -->
-<!--   <gazebo reference="panda_link0">
-  </gazebo> -->
   <gazebo reference="panda_link1">
     <mu1>0.2</mu1>
@@ -48,98 +45,4 @@
     <mu2>0.2</mu2>
   </gazebo>
-<!--   <gazebo reference="base_link">
-    <kp>10000.0</kp>
-    <kd>10.0</kd>
-    <mu1>0.1</mu1>
-    <mu2>0.1</mu2>
-    <fdir1>1 0 0</fdir1>
-    <maxVel>10.0</maxVel>
-    <minDepth>0.0005</minDepth>
-    <material>Gazebo/Grey</material>
-  </gazebo>
-  <gazebo reference="link_wheel_1">
-    <kp>500000.0</kp>
-    <kd>10.0</kd>
-    <mu1>10</mu1>
-    <mu2>10</mu2>
-    <fdir1>1 0 0</fdir1>
-    <maxVel>1.0</maxVel>
-    <minDepth>0.003</minDepth>
-    <material>Gazebo/Grey</material>
-  </gazebo>
-  <gazebo reference="link_wheel_2">
-    <kp>500000.0</kp>
-    <kd>10.0</kd>
-    <mu1>10</mu1>
-    <mu2>10</mu2>
-    <fdir1>1 0 0</fdir1>
-    <maxVel>1.0</maxVel>
-    <minDepth>0.003</minDepth>
-    <material>Gazebo/Grey</material>
-  </gazebo>
-  <gazebo reference="link_wheel_3">
-    <kp>500000.0</kp>
-    <kd>10.0</kd>
-    <mu1>10</mu1>
-    <mu2>10</mu2>
-    <fdir1>1 0 0</fdir1>
-    <maxVel>1.0</maxVel>
-    <minDepth>0.003</minDepth>
-    <material>Gazebo/Grey</material>
-  </gazebo>
-  <gazebo reference="joint_wheel_1">
-    <implicitSpringDamper>1</implicitSpringDamper>
-  </gazebo>
-  <gazebo reference="joint_wheel_2">
-    <implicitSpringDamper>1</implicitSpringDamper>
-  </gazebo>
-  <gazebo reference="joint_wheel_3">
-    <implicitSpringDamper>1</implicitSpringDamper>
-  </gazebo>
-  <gazebo reference="link_lift">
-    <material>Gazebo/White</material>
-  </gazebo>
-  <gazebo reference="link_waist">
-    <material>Gazebo/Orange</material>
-  </gazebo>
-  <gazebo reference="link_big_arm">
-    <material>Gazebo/White</material>
-  </gazebo>
-  <gazebo reference="link_forearm">
-    <material>Gazebo/Orange</material>
-  </gazebo>
-  <gazebo reference="link_wrist_pitching">
-    <material>Gazebo/White</material>
-  </gazebo>
-  <gazebo reference="link_wrist_rotation">
-    <material>Gazebo/White</material>
-  </gazebo>
-  <gazebo reference="link_finger_left">
-    <kp>1000000.0</kp>
-    <kd>100.0</kd>
-    <mu1>30.0</mu1>
-    <mu2>30.0</mu2>
-    <maxVel>1.0</maxVel>
-    <minDepth>0.001</minDepth>
-    <material>Gazebo/Orange</material>
-  </gazebo>
-  <gazebo reference="link_finger_right">
-    <kp>1000000.0</kp>
-    <kd>100.0</kd>
-    <mu1>30.0</mu1>
-    <mu2>30.0</mu2>
-    <maxVel>1.0</maxVel>
-    <minDepth>0.001</minDepth>
-    <material>Gazebo/Orange</material>
-  </gazebo>
-  <gazebo reference="link_gripper_frame">
-    <material>Gazebo/White</material>
-  </gazebo>
-  <gazebo reference="link_laser">
-    <material>Gazebo/Grey</material>
-  </gazebo>
-  <gazebo reference="link_kinect">
-    <material>Gazebo/Grey</material>
-  </gazebo> -->
 <!--   <gazebo reference="panda_hand">
     <sensor type="depth" name="kinect">

File: panda_description/urdf/hand.xacro (robot description, xacro)
@@ -20,9 +20,12 @@
         </geometry>
       </collision>
-<!--       <inertial>
-        <origin xyz="0 0 0.25" rpy="0 0 0" />
-        <mass value="0.5" />
-        <inertia ixx="1" ixy="0" ixz="0" iyy="1" iyz="0" izz="1" />
-      </inertial> -->
+      <inertial>
+        <origin xyz="-2.7600000000e-06 -6.1551000000e-04 2.3929520000e-02"
+                rpy="0 0 0" />
+        <mass value="2.36" />
+        <inertia ixx="8.0087281861e-03"  ixy="-1.3983247099e-06"
+                 ixz="3.1668653650e-07"  iyy="1.6099853693e-03"
+                 iyz="-1.4527159720e-04" izz="7.2469819837e-03" />
+      </inertial>
     </link>
     <link name="${ns}_leftfinger">
@@ -37,9 +40,12 @@
         </geometry>
       </collision>
-<!--       <inertial>
-        <origin xyz="0 0 0.25" rpy="0 0 0" />
-        <mass value="0.25" />
-        <inertia ixx="1" ixy="0" ixz="0" iyy="1" iyz="0" izz="1" />
-      </inertial> -->
+      <inertial>
+        <origin xyz="-2.4250000000e-05 1.1958490000e-02 2.3781550000e-02"
+                rpy="0 0 0" />
+        <mass value="0.73" />
+        <inertia ixx="1.9009821976e-04" ixy="-1.2251156196e-07"
+                 ixz="2.1231749953e-07" iyy="1.8154811386e-04"
+                 iyz="2.2800975511e-05" izz="5.5792802358e-05" />
+      </inertial>
     </link>
     <link name="${ns}_rightfinger">
@@ -56,9 +62,12 @@
         </geometry>
       </collision>
-<!--       <inertial>
-        <origin xyz="0 0 0.25" rpy="0 0 0" />
-        <mass value="0.25" />
-        <inertia ixx="1" ixy="0" ixz="0" iyy="1" iyz="0" izz="1" />
-      </inertial> -->
+      <inertial>
+        <origin xyz="-2.4250000000e-05 1.1958490000e-02 2.3781550000e-02"
+                rpy="0 0 0" />
+        <mass value="0.73" />
+        <inertia ixx="1.9009821976e-04" ixy="-1.2251156196e-07"
+                 ixz="2.1231749953e-07" iyy="1.8154811386e-04"
+                 iyz="2.2800975511e-05" izz="5.5792802358e-05" />
+      </inertial>
     </link>
     <joint name="${ns}_finger_joint1" type="prismatic">

File: panda_description/urdf/panda_arm.xacro (robot description, xacro)
@@ -21,7 +21,10 @@
       </collision>
       <inertial>
-        <origin xyz="0 0 0.05" rpy="0 0 0" />
-        <mass value="1" />
-        <inertia ixx="1" ixy="0" ixz="0" iyy="1" iyz="0" izz="1" />
+        <origin xyz="-2.9189750000e-02 -8.7947000000e-04 5.6603190000e-02"
+                rpy="0 0 0" />
+        <mass value="1.0" />
+        <inertia ixx="3.0208907507e-03"  ixy="-1.9469434530e-05"
+                 ixz="-4.5987519329e-04" iyy="3.9017274973e-03"
+                 iyz="-4.1208729424e-07" izz="4.0286070431e-03" />
       </inertial>
     </link>
@@ -38,7 +41,10 @@
       </collision>
       <inertial>
-        <origin xyz="0 0 -0.08" rpy="0 0 0" />
-        <mass value="1" />
-        <inertia ixx="1" ixy="0" ixz="0" iyy="1" iyz="0" izz="1" />
+        <origin xyz="1.1400000000e-05 -3.1265540000e-02 -6.9373290000e-02"
+                rpy="0 0 0" />
+        <mass value="1.0" />
+        <inertia ixx="5.9226730485e-03" ixy="1.4245315766e-07"
+                 ixz="3.8568507530e-07" iyy="5.1298138460e-03"
+                 iyz="1.1560796647e-03" izz="2.3931512155e-03" />
       </inertial>
     </link>
@@ -63,9 +69,10 @@
       </collision>
       <inertial>
-        <origin xyz="0 -0.05 0" rpy="0 0 0" />
-        <mass value="1" />
-        <inertia ixx="-1" ixy="0" ixz="0"
-                 iyy="-1" iyz="0"
-                 izz="-1" />
+        <origin xyz="-1.3180000000e-05 -7.0321540000e-02 3.1178270000e-02"
+                rpy="0 0 0" />
+        <mass value="1.0" />
+        <inertia ixx="5.9962199438e-03"  ixy="-6.7615014029e-07"
+                 ixz="-2.3493516929e-07" iyy="2.3948403893e-03"
+                 iyz="-1.1636087632e-03" izz="5.2033249732e-03" />
       </inertial>
     </link>
@@ -89,9 +96,12 @@
         </geometry>
       </collision>
-<!--       <inertial>
-        <origin xyz="0 0 0" rpy="0 0 0" />
-        <mass value="1" />
-        <inertia ixx="1" ixy="0" ixz="0" iyy="1" iyz="0" izz="1" />
-      </inertial> -->
+      <inertial>
+        <origin xyz="4.4348280000e-02 2.4928320000e-02 -3.8130030000e-02"
+                rpy="0 0 0" />
+        <mass value="0.78" />
+        <inertia ixx="2.4814391703e-03"  ixy="-4.8315843437e-04"
+                 ixz="-8.2557114619e-04" iyy="2.9935310139e-03"
+                 iyz="-4.4604815446e-04" izz="2.5083810118e-03" />
+      </inertial>
     </link>
     <joint name="${arm_id}_joint3" type="revolute">
@@ -114,9 +124,12 @@
         </geometry>
       </collision>
-<!--       <inertial>
-        <origin xyz="0 0 0.5" rpy="0 0 0" />
-        <mass value="1" />
-        <inertia ixx="1" ixy="0" ixz="0" iyy="1" iyz="0" izz="1" />
-      </inertial> -->
+      <inertial>
+        <origin xyz="-3.8550270000e-02 3.9525550000e-02 2.4716210000e-02"
+                rpy="0 0 0" />
+        <mass value="0.79" />
+        <inertia ixx="2.5698770428e-03"  ixy="8.5226293644e-04"
+                 ixz="-4.8914733021e-04" iyy="2.5435632961e-03"
+                 iyz="4.6078342421e-04"  izz="3.0898802746e-03" />
+      </inertial>
     </link>
     <joint name="${arm_id}_joint4" type="revolute">
@@ -139,9 +152,12 @@
         </geometry>
       </collision>
-<!--       <inertial>
-        <origin xyz="0 0 0.5" rpy="0 0 0" />
-        <mass value="1" />
-        <inertia ixx="1" ixy="0" ixz="0" iyy="1" iyz="0" izz="1" />
-      </inertial> -->
+      <inertial>
+        <origin xyz="-6.3700000000e-05 3.8412360000e-02 -1.0997013000e-01"
+                rpy="0 0 0" />
+        <mass value="1.14" />
+        <inertia ixx="9.9489526162e-03"  ixy="-3.0923971423e-06"
+                 ixz="-1.3276013105e-05" iyy="9.0449844181e-03"
+                 iyz="-1.9558597152e-03" izz="2.5774715454e-03" />
+      </inertial>
     </link>
     <joint name="${arm_id}_joint5" type="revolute">
@@ -164,9 +180,12 @@
         </geometry>
       </collision>
-<!--       <inertial>
-        <origin xyz="0 0 0.5" rpy="0 0 0" />
-        <mass value="1" />
-        <inertia ixx="1" ixy="0" ixz="0" iyy="1" iyz="0" izz="1" />
-      </inertial> -->
+      <inertial>
+        <origin xyz="5.1002280000e-02 6.9326700000e-03 6.1689700000e-03"
+                rpy="0 0 0" />
+        <mass value="0.48" />
+        <inertia ixx="7.7550750204e-04" ixy="-5.4535229445e-05"
+                 ixz="9.8447394353e-05" iyy="1.1843242027e-03"
+                 iyz="9.7507874688e-06" izz="1.4430443083e-03" />
+      </inertial>
     </link>
     <joint name="${arm_id}_joint6" type="revolute">
@@ -189,9 +208,12 @@
         </geometry>
       </collision>
-<!--       <inertial>
-        <origin xyz="0 0 0.5" rpy="0 0 0" />
-        <mass value="1" />
-        <inertia ixx="1" ixy="0" ixz="0" iyy="1" iyz="0" izz="1" />
-      </inertial> -->
+      <inertial>
+        <origin xyz="1.0361390000e-02 1.0359650000e-02 7.9107730000e-02"
+                rpy="0 0 0" />
+        <mass value="1.49" />
+        <inertia ixx="1.4440550235e-03"  ixy="-4.4171751527e-04"
+                 ixz="-4.8331020139e-05" iyy="1.4430197316e-03"
+                 iyz="-4.8495088634e-05" izz="2.2729277029e-03" />
+      </inertial>
     </link>
     <joint name="${arm_id}_joint7" type="revolute">
