Commit message: Format the package

File: panda_description/gazebo/panda_arm_hand_ros_control.xacro (robot description, xacro)
@@ -1,4 +1,4 @@
 <?xml version="1.0" encoding="utf-8"?>
-<robot xmlns:xacro="http://www.ros.org/wiki/xacro">
+<robot name="panda" xmlns:xacro="http://www.ros.org/wiki/xacro">
   <gazebo>
     <plugin name="gazebo_ros_control" filename="libgazebo_ros_control.so">

File: panda_description/gazebo/panda_arm_hand_transmission.xacro (robot description, xacro)
@@ -1,90 +1,90 @@
 <?xml version="1.0" encoding="utf-8"?>
-<robot xmlns:xacro="http://www.ros.org/wiki/xacro">
-  <transmission name="joint1_simp_trans">
+<robot name="panda" xmlns:xacro="http://www.ros.org/wiki/xacro">
+  <transmission name="joint_arm_1_simp_trans">
     <type>transmission_interface/SimpleTransmission</type>
-    <joint name="panda_joint1">
+    <joint name="joint_arm_1">
       <hardwareInterface>hardware_interface/PositionJointInterface</hardwareInterface>
     </joint>
-    <actuator name="joint1_actuator">
+    <actuator name="joint_arm_1_actuator">
       <hardwareInterface>hardware_interface/PositionJointInterface</hardwareInterface>
       <mechanicalReduction>1</mechanicalReduction>
     </actuator>
   </transmission>
-  <transmission name="joint2_simp_trans">
+  <transmission name="joint_arm_2_simp_trans">
     <type>transmission_interface/SimpleTransmission</type>
-    <joint name="panda_joint2">
+    <joint name="joint_arm_2">
       <hardwareInterface>hardware_interface/PositionJointInterface</hardwareInterface>
     </joint>
-    <actuator name="joint2_actuator">
+    <actuator name="joint_arm_2_actuator">
       <hardwareInterface>hardware_interface/PositionJointInterface</hardwareInterface>
       <mechanicalReduction>1</mechanicalReduction>
     </actuator>
   </transmission>
-  <transmission name="joint3_simp_trans">
+  <transmission name="joint_arm_3_simp_trans">
     <type>transmission_interface/SimpleTransmission</type>
-    <joint name="panda_joint3">
+    <joint name="joint_arm_3">
       <hardwareInterface>hardware_interface/PositionJointInterface</hardwareInterface>
     </joint>
-    <actuator name="joint3_actuator">
+    <actuator name="joint_arm_3_actuator">
       <hardwareInterface>hardware_interface/PositionJointInterface</hardwareInterface>
       <mechanicalReduction>1</mechanicalReduction>
     </actuator>
   </transmission>
-  <transmission name="joint4_simp_trans">
+  <transmission name="joint_arm_4_simp_trans">
     <type>transmission_interface/SimpleTransmission</type>
-    <joint name="panda_joint4">
+    <joint name="joint_arm_4">
       <hardwareInterface>hardware_interface/PositionJointInterface</hardwareInterface>
     </joint>
-    <actuator name="joint4_actuator">
+    <actuator name="joint_arm_4_actuator">
       <hardwareInterface>hardware_interface/PositionJointInterface</hardwareInterface>
       <mechanicalReduction>1</mechanicalReduction>
     </actuator>
   </transmission>
-  <transmission name="joint5_simp_trans">
+  <transmission name="joint_arm_5_simp_trans">
     <type>transmission_interface/SimpleTransmission</type>
-    <joint name="panda_joint5">
+    <joint name="joint_arm_5">
       <hardwareInterface>hardware_interface/PositionJointInterface</hardwareInterface>
     </joint>
-    <actuator name="joint5_actuator">
+    <actuator name="joint_arm_5_actuator">
       <hardwareInterface>hardware_interface/PositionJointInterface</hardwareInterface>
       <mechanicalReduction>1</mechanicalReduction>
     </actuator>
   </transmission>
-  <transmission name="joint6_simp_trans">
+  <transmission name="joint_arm_6_simp_trans">
     <type>transmission_interface/SimpleTransmission</type>
-    <joint name="panda_joint6">
+    <joint name="joint_arm_6">
       <hardwareInterface>hardware_interface/PositionJointInterface</hardwareInterface>
     </joint>
-    <actuator name="joint6_actuator">
+    <actuator name="joint_arm_6_actuator">
       <hardwareInterface>hardware_interface/PositionJointInterface</hardwareInterface>
       <mechanicalReduction>1</mechanicalReduction>
     </actuator>
   </transmission>
-  <transmission name="joint7_simp_trans">
+  <transmission name="joint_arm_7_simp_trans">
     <type>transmission_interface/SimpleTransmission</type>
-    <joint name="panda_joint7">
+    <joint name="joint_arm_7">
       <hardwareInterface>hardware_interface/PositionJointInterface</hardwareInterface>
     </joint>
-    <actuator name="joint7_actuator">
+    <actuator name="joint_arm_7_actuator">
       <hardwareInterface>hardware_interface/PositionJointInterface</hardwareInterface>
       <mechanicalReduction>1</mechanicalReduction>
     </actuator>
   </transmission>
-  <transmission name="finger_joint1_simp_trans">
+  <transmission name="joint_finger_l_simp_trans">
     <type>transmission_interface/SimpleTransmission</type>
-    <joint name="panda_finger_joint1">
+    <joint name="joint_finger_l">
       <hardwareInterface>hardware_interface/PositionJointInterface</hardwareInterface>
     </joint>
-    <actuator name="finger_joint1_actuator">
+    <actuator name="fjoint_finger_l_actuator">
       <hardwareInterface>hardware_interface/PositionJointInterface</hardwareInterface>
       <mechanicalReduction>1</mechanicalReduction>
     </actuator>
   </transmission>
-  <transmission name="finger_joint2_simp_trans">
+  <transmission name="joint_finger_r_simp_trans">
     <type>transmission_interface/SimpleTransmission</type>
-    <joint name="panda_finger_joint2">
+    <joint name="joint_finger_r">
       <hardwareInterface>hardware_interface/PositionJointInterface</hardwareInterface>
     </joint>
-    <actuator name="finger_joint2_actuator">
+    <actuator name="joint_finger_r_actuator">
       <hardwareInterface>hardware_interface/PositionJointInterface</hardwareInterface>
       <mechanicalReduction>1</mechanicalReduction>

File: panda_description/gazebo/panda_arm_hand_urdf.xacro (robot description, xacro)
@@ -1,6 +1,6 @@
 <?xml version="1.0" encoding="utf-8"?>
-<robot xmlns:xacro="http://www.ros.org/wiki/xacro">
+<robot name="panda" xmlns:xacro="http://www.ros.org/wiki/xacro">
 <xacro:property name="M_PI" value="3.1415926535897931" />
-  <gazebo reference="panda_link0">
+  <gazebo reference="link_arm_0">
     <kp>1000000.0</kp>
     <kd>100.0</kd>
@@ -8,5 +8,5 @@
     <mu2>30.0</mu2>
   </gazebo>
-  <gazebo reference="panda_link1">
+  <gazebo reference="link_arm_1">
     <kp>1000000.0</kp>
     <kd>100.0</kd>
@@ -14,5 +14,5 @@
     <mu2>30.0</mu2>
   </gazebo>
-  <gazebo reference="panda_link2">
+  <gazebo reference="link_arm_2">
     <kp>1000000.0</kp>
     <kd>100.0</kd>
@@ -20,5 +20,5 @@
     <mu2>30.0</mu2>
   </gazebo>
-  <gazebo reference="panda_link3">
+  <gazebo reference="link_arm_3">
     <kp>1000000.0</kp>
     <kd>100.0</kd>
@@ -26,5 +26,5 @@
     <mu2>30.0</mu2>
   </gazebo>
-  <gazebo reference="panda_link4">
+  <gazebo reference="link_arm_4">
     <kp>1000000.0</kp>
     <kd>100.0</kd>
@@ -32,5 +32,5 @@
     <mu2>30.0</mu2>
   </gazebo>
-  <gazebo reference="panda_link5">
+  <gazebo reference="link_arm_5">
     <kp>1000000.0</kp>
     <kd>100.0</kd>
@@ -38,5 +38,5 @@
     <mu2>30.0</mu2>
   </gazebo>
-  <gazebo reference="panda_link6">
+  <gazebo reference="link_arm_6">
     <kp>1000000.0</kp>
     <kd>100.0</kd>
@@ -44,5 +44,5 @@
     <mu2>30.0</mu2>
   </gazebo>
-  <gazebo reference="panda_link7">
+  <gazebo reference="link_arm_7">
     <kp>1000000.0</kp>
     <kd>100.0</kd>
@@ -50,5 +50,5 @@
     <mu2>30.0</mu2>
   </gazebo>
-  <gazebo reference="panda_link8">
+  <gazebo reference="link_hand">
     <kp>1000000.0</kp>
     <kd>100.0</kd>
@@ -56,5 +56,5 @@
     <mu2>30.0</mu2>
   </gazebo>
-  <gazebo reference="panda_hand">
+  <gazebo reference="link_finger_l">
     <kp>1000000.0</kp>
     <kd>100.0</kd>
@@ -62,5 +62,5 @@
     <mu2>30.0</mu2>
   </gazebo>
-  <gazebo reference="panda_leftfinger">
+  <gazebo reference="link_finger_r">
     <kp>1000000.0</kp>
     <kd>100.0</kd>
@@ -68,10 +68,5 @@
     <mu2>30.0</mu2>
   </gazebo>
-  <gazebo reference="panda_rightfinger">
-    <kp>1000000.0</kp>
-    <kd>100.0</kd>
-    <mu1>30.0</mu1>
-    <mu2>30.0</mu2>
-  </gazebo>
+<!--
   <gazebo reference="panda_hand">
     <sensor type="depth" name="kinect">
@@ -113,4 +108,4 @@
       </plugin>
     </sensor>
-  </gazebo>
+  </gazebo> -->
 </robot>

File: panda_description/urdf/panda_arm.urdf.xacro (robot description, xacro)
@@ -1,5 +1,4 @@
 <?xml version='1.0' encoding='utf-8'?>
-<robot xmlns:xacro="http://www.ros.org/wiki/xacro" name="panda">
+<robot name="panda_arm" xmlns:xacro="http://www.ros.org/wiki/xacro" >
   <xacro:include filename="$(find panda_description)/urdf/panda_arm.xacro" />
-  <xacro:panda_arm />
 </robot>

File: panda_description/urdf/panda_arm.xacro (robot description, xacro)
@@ -1,21 +1,22 @@
 <?xml version='1.0' encoding='utf-8'?>
-<robot xmlns:xacro="http://www.ros.org/wiki/xacro" name="panda">
-  <xacro:macro name="panda_arm" params="arm_id:='panda' description_pkg:='panda_description' connected_to:='' xyz:='0 0 0' rpy:='0 0 0'">
-    <xacro:unless value="${not connected_to}">
-      <joint name="${arm_id}_joint_${connected_to}" type="fixed">
-        <parent link="${connected_to}" />
-        <child link="${arm_id}_link0" />
-        <origin rpy="${rpy}" xyz="${xyz}" />
-      </joint>
-    </xacro:unless>
-    <link name="${arm_id}_link0">
-      <visual>
-        <geometry>
-          <mesh filename="package://${description_pkg}/meshes/visual/link0.dae" />
-        </geometry>
-      </visual>
-      <collision>
-        <geometry>
-          <mesh filename="package://${description_pkg}/meshes/collision/link0.stl" />
+<robot name="panda_arm" xmlns:xacro="http://www.ros.org/wiki/xacro">
+  <xacro:macro name="panda_arm" params="name:='arm' xyz:='0 0 0' rpy:='0 0 0'">
+    <link name="link_${name}_base" />
+<!--       <visual>
+        <origin xyz="${xyz}" rpy="${rpy}" />
+        <geometry>
+          <box size="0.05 0.05 0.05" />
+        </geometry>
+      </visual>
+    </link> -->
+    <link name="link_${name}_0">
+      <visual>
+        <geometry>
+          <mesh filename="package://panda_description/meshes/visual/link0.dae" />
+        </geometry>
+      </visual>
+      <collision>
+        <geometry>
+          <mesh filename="package://panda_description/meshes/collision/link0.stl" />
         </geometry>
       </collision>
@@ -29,13 +30,18 @@
       </inertial>
     </link>
-    <link name="${arm_id}_link1">
-      <visual>
-        <geometry>
-          <mesh filename="package://${description_pkg}/meshes/visual/link1.dae" />
-        </geometry>
-      </visual>
-      <collision>
-        <geometry>
-          <mesh filename="package://${description_pkg}/meshes/collision/link1.stl" />
+    <joint name="$joint_${name}_base" type="fixed">
+      <origin xyz="${xyz}" rpy="${rpy}" />
+      <parent link="link_${name}_base" />
+      <child  link="link_${name}_0" />
+    </joint>
+    <link name="link_${name}_1">
+      <visual>
+        <geometry>
+          <mesh filename="package://panda_description/meshes/visual/link1.dae" />
+        </geometry>
+      </visual>
+      <collision>
+        <geometry>
+          <mesh filename="package://panda_description/meshes/collision/link1.stl" />
         </geometry>
       </collision>
@@ -49,21 +55,21 @@
       </inertial>
     </link>
-    <joint name="${arm_id}_joint1" type="revolute">
-      <safety_controller k_position="100.0" k_velocity="40.0" soft_lower_limit="-2.8973" soft_upper_limit="2.8973" />
+    <joint name="joint_${name}_1" type="revolute">
       <origin rpy="0 0 0" xyz="0 0 0.333" />
-      <parent link="${arm_id}_link0" />
-      <child link="${arm_id}_link1" />
+      <parent link="link_${name}_0" />
+      <child link="link_${name}_1" />
       <axis xyz="0 0 1" />
       <limit effort="87" lower="-2.9671" upper="2.9671" velocity="2.3925" />
-    </joint>
-    <link name="${arm_id}_link2">
-      <visual>
-        <geometry>
-          <mesh filename="package://${description_pkg}/meshes/visual/link2.dae" />
-        </geometry>
-      </visual>
-      <collision>
-        <geometry>
-          <mesh filename="package://${description_pkg}/meshes/collision/link2.stl" />
+      <safety_controller k_position="100.0" k_velocity="40.0" soft_lower_limit="-2.8973" soft_upper_limit="2.8973" />
+    </joint>
+    <link name="link_${name}_2">
+      <visual>
+        <geometry>
+          <mesh filename="package://panda_description/meshes/visual/link2.dae" />
+        </geometry>
+      </visual>
+      <collision>
+        <geometry>
+          <mesh filename="package://panda_description/meshes/collision/link2.stl" />
         </geometry>
       </collision>
@@ -77,21 +83,21 @@
       </inertial>
     </link>
-    <joint name="${arm_id}_joint2" type="revolute">
+    <joint name="joint_${name}_2" type="revolute">
+      <origin rpy="${-pi/2} 0 0" xyz="0 0 0" />
+      <parent link="link_${name}_1" />
+      <child link="link_${name}_2" />
+      <axis xyz="0 0 1" />
+      <limit effort="87" lower="-1.8326" upper="1.8326" velocity="2.3925" />
       <safety_controller k_position="100.0" k_velocity="40.0" soft_lower_limit="-1.7628" soft_upper_limit="1.7628" />
-      <origin rpy="${-pi/2} 0 0" xyz="0 0 0" />
-      <parent link="${arm_id}_link1" />
-      <child link="${arm_id}_link2" />
-      <axis xyz="0 0 1" />
-      <limit effort="87" lower="-1.8326" upper="1.8326" velocity="2.3925" />
-    </joint>
-    <link name="${arm_id}_link3">
-      <visual>
-        <geometry>
-          <mesh filename="package://${description_pkg}/meshes/visual/link3.dae"/>
-        </geometry>
-      </visual>
-      <collision>
-        <geometry>
-          <mesh filename="package://${description_pkg}/meshes/collision/link3.stl" />
+    </joint>
+    <link name="link_${name}_3">
+      <visual>
+        <geometry>
+          <mesh filename="package://panda_description/meshes/visual/link3.dae"/>
+        </geometry>
+      </visual>
+      <collision>
+        <geometry>
+          <mesh filename="package://panda_description/meshes/collision/link3.stl" />
         </geometry>
       </collision>
@@ -105,21 +111,21 @@
       </inertial>
     </link>
-    <joint name="${arm_id}_joint3" type="revolute">
-      <safety_controller k_position="100.0" k_velocity="40.0" soft_lower_limit="-2.8973" soft_upper_limit="2.8973" />
+    <joint name="joint_${name}_3" type="revolute">
       <origin rpy="${pi/2} 0 0" xyz="0 -0.316 0" />
-      <parent link="${arm_id}_link2" />
-      <child link="${arm_id}_link3" />
+      <parent link="link_${name}_2" />
+      <child link="link_${name}_3" />
       <axis xyz="0 0 1" />
       <limit effort="87" lower="-2.9671" upper="2.9671" velocity="2.3925" />
-    </joint>
-    <link name="${arm_id}_link4">
-      <visual>
-        <geometry>
-          <mesh filename="package://${description_pkg}/meshes/visual/link4.dae" />
-        </geometry>
-      </visual>
-      <collision>
-        <geometry>
-          <mesh filename="package://${description_pkg}/meshes/collision/link4.stl" />
+      <safety_controller k_position="100.0" k_velocity="40.0" soft_lower_limit="-2.8973" soft_upper_limit="2.8973" />
+    </joint>
+    <link name="link_${name}_4">
+      <visual>
+        <geometry>
+          <mesh filename="package://panda_description/meshes/visual/link4.dae" />
+        </geometry>
+      </visual>
+      <collision>
+        <geometry>
+          <mesh filename="package://panda_description/meshes/collision/link4.stl" />
         </geometry>
       </collision>
@@ -133,21 +139,22 @@
       </inertial>
     </link>
-    <joint name="${arm_id}_joint4" type="revolute">
+    <joint name="joint_${name}_4" type="revolute">
       <safety_controller k_position="100.0" k_velocity="40.0" soft_lower_limit="-3.0718" soft_upper_limit="0.0175" />
       <origin rpy="${pi/2} 0 0" xyz="0.0825 0 0" />
-      <parent link="${arm_id}_link3" />
-      <child link="${arm_id}_link4" />
+      <parent link="link_${name}_3" />
+      <child link="link_${name}_4" />
       <axis xyz="0 0 1" />
       <limit effort="87" lower="-3.1416" upper="0.0873" velocity="2.3925" />
-    </joint>
-    <link name="${arm_id}_link5">
-      <visual>
-        <geometry>
-          <mesh filename="package://${description_pkg}/meshes/visual/link5.dae" />
-        </geometry>
-      </visual>
-      <collision>
-        <geometry>
-          <mesh filename="package://${description_pkg}/meshes/collision/link5.stl" />
+      <safety_controller k_position="100.0" k_velocity="40.0" soft_lower_limit="-3.0718" soft_upper_limit="0.0175" />
+    </joint>
+    <link name="link_${name}_5">
+      <visual>
+        <geometry>
+          <mesh filename="package://panda_description/meshes/visual/link5.dae" />
+        </geometry>
+      </visual>
+      <collision>
+        <geometry>
+          <mesh filename="package://panda_description/meshes/collision/link5.stl" />
         </geometry>
       </collision>
@@ -161,21 +168,21 @@
       </inertial>
     </link>
-    <joint name="${arm_id}_joint5" type="revolute">
-      <safety_controller k_position="100.0" k_velocity="40.0" soft_lower_limit="-2.8973" soft_upper_limit="2.8973" />
+    <joint name="joint_${name}_5" type="revolute">
       <origin rpy="${-pi/2} 0 0" xyz="-0.0825 0.384 0" />
-      <parent link="${arm_id}_link4" />
-      <child link="${arm_id}_link5" />
+      <parent link="link_${name}_4" />
+      <child link="link_${name}_5" />
       <axis xyz="0 0 1" />
       <limit effort="12" lower="-2.9671" upper="2.9671" velocity="2.8710" />
-    </joint>
-    <link name="${arm_id}_link6">
-      <visual>
-        <geometry>
-          <mesh filename="package://${description_pkg}/meshes/visual/link6.dae" />
-        </geometry>
-      </visual>
-      <collision>
-        <geometry>
-          <mesh filename="package://${description_pkg}/meshes/collision/link6.stl" />
+      <safety_controller k_position="100.0" k_velocity="40.0" soft_lower_limit="-2.8973" soft_upper_limit="2.8973" />
+    </joint>
+    <link name="link_${name}_6">
+      <visual>
+        <geometry>
+          <mesh filename="package://panda_description/meshes/visual/link6.dae" />
+        </geometry>
+      </visual>
+      <collision>
+        <geometry>
+          <mesh filename="package://panda_description/meshes/collision/link6.stl" />
         </geometry>
       </collision>
@@ -189,21 +196,21 @@
       </inertial>
     </link>
-    <joint name="${arm_id}_joint6" type="revolute">
+    <joint name="joint_${name}_6" type="revolute">
+      <origin rpy="${pi/2} 0 0" xyz="0 0 0" />
+      <parent link="link_${name}_5" />
+      <child link="link_${name}_6" />
+      <axis xyz="0 0 1" />
+      <limit effort="12" lower="-0.0873" upper="3.8223" velocity="2.8710" />
       <safety_controller k_position="100.0" k_velocity="40.0" soft_lower_limit="-0.0175" soft_upper_limit="3.7525" />
-      <origin rpy="${pi/2} 0 0" xyz="0 0 0" />
-      <parent link="${arm_id}_link5" />
-      <child link="${arm_id}_link6" />
-      <axis xyz="0 0 1" />
-      <limit effort="12" lower="-0.0873" upper="3.8223" velocity="2.8710" />
-    </joint>
-    <link name="${arm_id}_link7">
-      <visual>
-        <geometry>
-          <mesh filename="package://${description_pkg}/meshes/visual/link7.dae" />
-        </geometry>
-      </visual>
-      <collision>
-        <geometry>
-          <mesh filename="package://${description_pkg}/meshes/collision/link7.stl" />
+    </joint>
+    <link name="link_${name}_7">
+      <visual>
+        <geometry>
+          <mesh filename="package://panda_description/meshes/visual/link7.dae" />
+        </geometry>
+      </visual>
+      <collision>
+        <geometry>
+          <mesh filename="package://panda_description/meshes/collision/link7.stl" />
         </geometry>
       </collision>
@@ -217,17 +224,17 @@
       </inertial>
     </link>
-    <joint name="${arm_id}_joint7" type="revolute">
-      <safety_controller k_position="100.0" k_velocity="40.0" soft_lower_limit="-2.8973" soft_upper_limit="2.8973" />
+    <joint name="joint_${name}_7" type="revolute">
       <origin rpy="${pi/2} 0 0" xyz="0.088 0 0" />
-      <parent link="${arm_id}_link6" />
-      <child link="${arm_id}_link7" />
+      <parent link="link_${name}_6" />
+      <child link="link_${name}_7" />
       <axis xyz="0 0 1" />
       <limit effort="12" lower="-2.9671" upper="2.9671" velocity="2.8710" />
-    </joint>
-    <link name="${arm_id}_link8" />
-    <joint name="${arm_id}_joint8" type="fixed">
+      <safety_controller k_position="100.0" k_velocity="40.0" soft_lower_limit="-2.8973" soft_upper_limit="2.8973" />
+    </joint>
+    <link name="link_${name}_8" />
+    <joint name="joint_${name}_8" type="fixed">
       <origin rpy="0 0 0" xyz="0 0 0.107" />
-      <parent link="${arm_id}_link7" />
-      <child link="${arm_id}_link8" />
+      <parent link="link_${name}_7" />
+      <child link="link_${name}_8" />
       <axis xyz="0 0 0" />
     </joint>

File: panda_description/urdf/panda_arm_hand.urdf.xacro (robot description, xacro)
@@ -1,7 +1,7 @@
 <?xml version="1.0" encoding="utf-8"?>
-<robot xmlns:xacro="http://www.ros.org/wiki/xacro" name="panda">
+<robot name="panda" xmlns:xacro="http://www.ros.org/wiki/xacro">
   <xacro:include filename="$(find panda_description)/urdf/panda_arm.xacro" />
-  <xacro:include filename="$(find panda_description)/urdf/hand.xacro" />
+  <xacro:include filename="$(find panda_description)/urdf/panda_hand.xacro" />
   <xacro:panda_arm />
-  <xacro:hand ns="panda" rpy="0 0 ${-pi/4}" connected_to="panda_link8" />
+  <xacro:panda_hand rpy="0 0 ${-pi/4}" />
 </robot>
