Commit message: Format the package

File: panda_description/urdf/panda_hand.xacro (robot description, xacro)
@@ -1,13 +1,6 @@
 <?xml version="1.0" encoding="utf-8"?>
-<robot xmlns:xacro="http://www.ros.org/wiki/xacro" name="hand">
-  <xacro:macro name="hand" params="connected_to:='' ns:='' rpy:='0 0 0' xyz:='0 0 0' ">
-    <xacro:unless value="${connected_to == ''}">
-      <joint name="${ns}_hand_joint" type="fixed">
-        <parent link="${connected_to}" />
-        <child link="${ns}_hand" />
-        <origin xyz="${xyz}" rpy="${rpy}" />
-      </joint>
-    </xacro:unless>
-    <link name="${ns}_hand">
+<robot name="panda_hand" xmlns:xacro="http://www.ros.org/wiki/xacro">
+  <xacro:macro name="panda_hand" params="name:='hand' parent:='link_arm_8'  rpy:='0 0 0' xyz:='0 0 0'">
+    <link name="link_${name}">
       <visual>
         <geometry>
@@ -29,5 +22,10 @@
       </inertial>
     </link>
-    <link name="${ns}_leftfinger">
+    <joint name="joint_${name}" type="fixed">
+      <origin xyz="${xyz}" rpy="${rpy}" />
+      <parent link="${parent}" />
+      <child link="link_${name}" />
+    </joint>
+    <link name="link_finger_l">
       <visual>
         <geometry>
@@ -49,5 +47,5 @@
       </inertial>
     </link>
-    <link name="${ns}_rightfinger">
+    <link name="link_finger_r">
       <visual>
         <origin xyz="0 0 0" rpy="0 0 ${pi}" />
@@ -71,18 +69,18 @@
       </inertial>
     </link>
-    <joint name="${ns}_finger_joint1" type="prismatic">
-      <parent link="${ns}_hand" />
-      <child link="${ns}_leftfinger" />
+    <joint name="joint_finger_l" type="prismatic">
+      <parent link="link_${name}" />
+      <child link="link_finger_l" />
       <origin xyz="0 0 0.0584" rpy="0 0 0" />
       <axis xyz="0 1 0" />
       <limit effort="20" lower="0.0" upper="0.04" velocity="0.2" />
     </joint>
-    <joint name="${ns}_finger_joint2" type="prismatic">
-      <parent link="${ns}_hand" />
-      <child link="${ns}_rightfinger" />
+    <joint name="joint_finger_r" type="prismatic">
+      <parent link="link_${name}" />
+      <child link="link_finger_r" />
       <origin xyz="0 0 0.0584" rpy="0 0 0" />
       <axis xyz="0 -1 0" />
       <limit effort="20" lower="0.0" upper="0.04" velocity="0.2" />
-      <mimic joint="${ns}_finger_joint1" />
+      <mimic joint="joint_finger_l" />
     </joint>
   </xacro:macro>
