Commit message: Modify panda's xacro

File: panda_description/gazebo/panda_arm_hand_urdf.xacro (robot description, xacro)
@@ -2,62 +2,50 @@
 <robot xmlns:xacro="http://www.ros.org/wiki/xacro">
 <!-- <xacro:property name="M_PI" value="3.1415926535897931" /> -->
-<gazebo reference="panda_link0">
-  <material>Gazebo/Black</material>
-</gazebo>
-<gazebo reference="panda_link1">
-  <mu1>0.2</mu1>
-  <mu2>0.2</mu2>
-  <material>Gazebo/Orange</material>
-</gazebo>
-<gazebo reference="panda_link2">
-  <mu1>0.2</mu1>
-  <mu2>0.2</mu2>
-  <material>Gazebo/Orange</material>
-</gazebo>
-<gazebo reference="panda_link3">
-  <mu1>0.2</mu1>
-  <mu2>0.2</mu2>
-  <material>Gazebo/Orange</material>
-</gazebo>
-<gazebo reference="panda_link4">
-  <mu1>0.2</mu1>
-  <mu2>0.2</mu2>
-  <material>Gazebo/Orange</material>
-</gazebo>
-<gazebo reference="panda_link5">
-  <mu1>0.2</mu1>
-  <mu2>0.2</mu2>
-  <material>Gazebo/Orange</material>
-</gazebo>
-<gazebo reference="panda_link6">
-  <mu1>0.2</mu1>
-  <mu2>0.2</mu2>
-  <material>Gazebo/Orange</material>
-</gazebo>
-<gazebo reference="panda_link7">
-  <mu1>0.2</mu1>
-  <mu2>0.2</mu2>
-  <material>Gazebo/Orange</material>
-</gazebo>
-<gazebo reference="panda_link8">
-  <mu1>0.2</mu1>
-  <mu2>0.2</mu2>
-  <material>Gazebo/Orange</material>
-</gazebo>
-<gazebo reference="panda_hand">
-  <mu1>0.2</mu1>
-  <mu2>0.2</mu2>
-  <material>Gazebo/Orange</material>
-</gazebo>
-<gazebo reference="panda_leftfinger">
-  <mu1>0.2</mu1>
-  <mu2>0.2</mu2>
-  <material>Gazebo/Red</material>
-</gazebo>
-<gazebo reference="panda_rightfinger">
-  <mu1>0.2</mu1>
-  <mu2>0.2</mu2>
-  <material>Gazebo/Red</material>
-</gazebo>
+<!--   <gazebo reference="panda_link0">
+  </gazebo> -->
+  <gazebo reference="panda_link1">
+    <mu1>0.2</mu1>
+    <mu2>0.2</mu2>
+  </gazebo>
+  <gazebo reference="panda_link2">
+    <mu1>0.2</mu1>
+    <mu2>0.2</mu2>
+  </gazebo>
+  <gazebo reference="panda_link3">
+    <mu1>0.2</mu1>
+    <mu2>0.2</mu2>
+  </gazebo>
+  <gazebo reference="panda_link4">
+    <mu1>0.2</mu1>
+    <mu2>0.2</mu2>
+  </gazebo>
+  <gazebo reference="panda_link5">
+    <mu1>0.2</mu1>
+    <mu2>0.2</mu2>
+  </gazebo>
+  <gazebo reference="panda_link6">
+    <mu1>0.2</mu1>
+    <mu2>0.2</mu2>
+  </gazebo>
+  <gazebo reference="panda_link7">
+    <mu1>0.2</mu1>
+    <mu2>0.2</mu2>
+  </gazebo>
+  <gazebo reference="panda_link8">
+    <mu1>0.2</mu1>
+    <mu2>0.2</mu2>
+  </gazebo>
+  <gazebo reference="panda_hand">
+    <mu1>0.2</mu1>
+    <mu2>0.2</mu2>
+  </gazebo>
+  <gazebo reference="panda_leftfinger">
+    <mu1>0.2</mu1>
+    <mu2>0.2</mu2>
+  </gazebo>
+  <gazebo reference="panda_rightfinger">
+    <mu1>0.2</mu1>
+    <mu2>0.2</mu2>
+  </gazebo>
 <!--   <gazebo reference="base_link">
     <kp>10000.0</kp>

File: panda_description/urdf/panda_arm.xacro (robot description, xacro)
@@ -20,4 +20,9 @@
         </geometry>
       </collision>
+      <inertial>
+        <origin xyz="0 0 0" rpy="0 0 0" />
+        <mass value="1" />
+        <inertia ixx="0" ixy="0" ixz="0" iyy="0" iyz="0" izz="0" />
+      </inertial>
     </link>
     <link name="${arm_id}_link1">
@@ -32,4 +37,9 @@
         </geometry>
       </collision>
+      <inertial>
+        <origin xyz="0 0 0" rpy="0 0 0" />
+        <mass value="1" />
+        <inertia ixx="0" ixy="0" ixz="0" iyy="0" iyz="0" izz="0" />
+      </inertial>
     </link>
     <joint name="${arm_id}_joint1" type="revolute">
@@ -52,4 +62,9 @@
         </geometry>
       </collision>
+      <inertial>
+        <origin xyz="0 0 0" rpy="0 0 0" />
+        <mass value="1" />
+        <inertia ixx="0" ixy="0" ixz="0" iyy="0" iyz="0" izz="0" />
+      </inertial>
     </link>
     <joint name="${arm_id}_joint2" type="revolute">
@@ -72,4 +87,9 @@
         </geometry>
       </collision>
+      <inertial>
+        <origin xyz="0 0 0" rpy="0 0 0" />
+        <mass value="1" />
+        <inertia ixx="0" ixy="0" ixz="0" iyy="0" iyz="0" izz="0" />
+      </inertial>
     </link>
     <joint name="${arm_id}_joint3" type="revolute">
@@ -92,4 +112,9 @@
         </geometry>
       </collision>
+      <inertial>
+        <origin xyz="0 0 0" rpy="0 0 0" />
+        <mass value="1" />
+        <inertia ixx="0" ixy="0" ixz="0" iyy="0" iyz="0" izz="0" />
+      </inertial>
     </link>
     <joint name="${arm_id}_joint4" type="revolute">
@@ -112,4 +137,9 @@
         </geometry>
       </collision>
+      <inertial>
+        <origin xyz="0 0 0" rpy="0 0 0" />
+        <mass value="1" />
+        <inertia ixx="0" ixy="0" ixz="0" iyy="0" iyz="0" izz="0" />
+      </inertial>
     </link>
     <joint name="${arm_id}_joint5" type="revolute">
@@ -132,4 +162,9 @@
         </geometry>
       </collision>
+      <inertial>
+        <origin xyz="0 0 0" rpy="0 0 0" />
+        <mass value="1" />
+        <inertia ixx="0" ixy="0" ixz="0" iyy="0" iyz="0" izz="0" />
+      </inertial>
     </link>
     <joint name="${arm_id}_joint6" type="revolute">
@@ -152,4 +187,9 @@
         </geometry>
       </collision>
+      <inertial>
+        <origin xyz="0 0 0" rpy="0 0 0" />
+        <mass value="1" />
+        <inertia ixx="0" ixy="0" ixz="0" iyy="0" iyz="0" izz="0" />
+      </inertial>
     </link>
     <joint name="${arm_id}_joint7" type="revolute">

Commit message: Modify some files

File: panda_description/gazebo/panda_arm_hand_urdf.xacro (robot description, xacro)
@@ -1,49 +1,78 @@
 <?xml version="1.0" encoding="utf-8"?>
 <robot xmlns:xacro="http://www.ros.org/wiki/xacro">
+<xacro:property name="M_PI" value="3.1415926535897931" />
+  <gazebo reference="panda_link0">
+    <kp>1000000.0</kp>
+    <kd>100.0</kd>
+    <mu1>30.0</mu1>
+    <mu2>30.0</mu2>
+  </gazebo>
   <gazebo reference="panda_link1">
-    <mu1>0.2</mu1>
-    <mu2>0.2</mu2>
+    <kp>1000000.0</kp>
+    <kd>100.0</kd>
+    <mu1>30.0</mu1>
+    <mu2>30.0</mu2>
   </gazebo>
   <gazebo reference="panda_link2">
-    <mu1>0.2</mu1>
-    <mu2>0.2</mu2>
+    <kp>1000000.0</kp>
+    <kd>100.0</kd>
+    <mu1>30.0</mu1>
+    <mu2>30.0</mu2>
   </gazebo>
   <gazebo reference="panda_link3">
-    <mu1>0.2</mu1>
-    <mu2>0.2</mu2>
+    <kp>1000000.0</kp>
+    <kd>100.0</kd>
+    <mu1>30.0</mu1>
+    <mu2>30.0</mu2>
   </gazebo>
   <gazebo reference="panda_link4">
-    <mu1>0.2</mu1>
-    <mu2>0.2</mu2>
+    <kp>1000000.0</kp>
+    <kd>100.0</kd>
+    <mu1>30.0</mu1>
+    <mu2>30.0</mu2>
   </gazebo>
   <gazebo reference="panda_link5">
-    <mu1>0.2</mu1>
-    <mu2>0.2</mu2>
+    <kp>1000000.0</kp>
+    <kd>100.0</kd>
+    <mu1>30.0</mu1>
+    <mu2>30.0</mu2>
   </gazebo>
   <gazebo reference="panda_link6">
-    <mu1>0.2</mu1>
-    <mu2>0.2</mu2>
+    <kp>1000000.0</kp>
+    <kd>100.0</kd>
+    <mu1>30.0</mu1>
+    <mu2>30.0</mu2>
   </gazebo>
   <gazebo reference="panda_link7">
-    <mu1>0.2</mu1>
-    <mu2>0.2</mu2>
+    <kp>1000000.0</kp>
+    <kd>100.0</kd>
+    <mu1>30.0</mu1>
+    <mu2>30.0</mu2>
   </gazebo>
   <gazebo reference="panda_link8">
-    <mu1>0.2</mu1>
-    <mu2>0.2</mu2>
+    <kp>1000000.0</kp>
+    <kd>100.0</kd>
+    <mu1>30.0</mu1>
+    <mu2>30.0</mu2>
   </gazebo>
   <gazebo reference="panda_hand">
-    <mu1>0.2</mu1>
-    <mu2>0.2</mu2>
+    <kp>1000000.0</kp>
+    <kd>100.0</kd>
+    <mu1>30.0</mu1>
+    <mu2>30.0</mu2>
   </gazebo>
   <gazebo reference="panda_leftfinger">
-    <mu1>0.2</mu1>
-    <mu2>0.2</mu2>
+    <kp>1000000.0</kp>
+    <kd>100.0</kd>
+    <mu1>30.0</mu1>
+    <mu2>30.0</mu2>
   </gazebo>
   <gazebo reference="panda_rightfinger">
-    <mu1>0.2</mu1>
-    <mu2>0.2</mu2>
+    <kp>1000000.0</kp>
+    <kd>100.0</kd>
+    <mu1>30.0</mu1>
+    <mu2>30.0</mu2>
   </gazebo>
-<!--   <gazebo reference="panda_hand">
+  <gazebo reference="panda_hand">
     <sensor type="depth" name="kinect">
       <update_rate>20</update_rate>
@@ -84,4 +113,4 @@
       </plugin>
     </sensor>
-  </gazebo> -->
+  </gazebo>
 </robot>

Commit message: Add xtion module

File: panda_description/gazebo/panda_arm_hand_urdf.xacro (robot description, xacro)
@@ -1,5 +1,5 @@
 <?xml version="1.0" encoding="utf-8"?>
 <robot name="panda" xmlns:xacro="http://www.ros.org/wiki/xacro">
-<xacro:property name="M_PI" value="3.1415926535897931" />
+  <xacro:property name="deg_to_rad" value="0.01745329251994329577"/>
   <gazebo reference="link_arm_0">
     <kp>1000000.0</kp>
@@ -50,4 +50,10 @@
     <mu2>30.0</mu2>
   </gazebo>
+  <gazebo reference="link_arm_8">
+    <kp>1000000.0</kp>
+    <kd>100.0</kd>
+    <mu1>30.0</mu1>
+    <mu2>30.0</mu2>
+  </gazebo>
   <gazebo reference="link_hand">
     <kp>1000000.0</kp>
@@ -68,10 +74,10 @@
     <mu2>30.0</mu2>
   </gazebo>
-<!--
-  <gazebo reference="panda_hand">
-    <sensor type="depth" name="kinect">
+  <gazebo reference="link_xtion">
+    <sensor type="depth" name="xtion_sensor">
+      <always_on>true</always_on>
       <update_rate>20</update_rate>
       <camera>
-        <horizontal_fov>${60 * M_PI/180.0}</horizontal_fov>
+        <horizontal_fov>${60 * deg_to_rad}</horizontal_fov>
         <image>
           <format>R8G8B8</format>
@@ -84,15 +90,15 @@
         </clip>
       </camera>
-      <plugin name="kinect_controller" filename="libgazebo_ros_openni_kinect.so">
+      <plugin name="xtion_controller" filename="libgazebo_ros_openni_kinect.so">
         <baseline>0.1</baseline>
         <alwaysOn>true</alwaysOn>
         <updateRate>15.0</updateRate>
-        <cameraName>hand_kinect</cameraName>
-        <imageTopicName>/hand_kinect/rgb/image_raw</imageTopicName>
-        <cameraInfoTopicName>/hand_kinect/rgb/camera_info</cameraInfoTopicName>
-        <depthImageTopicName>/hand_kinect/depth/image_raw</depthImageTopicName>
-        <depthImageCameraInfoTopicName>/hand_kinect/depth/camera_info</depthImageCameraInfoTopicName>
-        <pointCloudTopicName>/hand_kinect/depth/points</pointCloudTopicName>
-        <frameName>panda_hand</frameName>
+        <cameraName>xtion_sensor</cameraName>
+        <imageTopicName>/xtion_sensor/rgb/image_raw</imageTopicName>
+        <cameraInfoTopicName>/xtion_sensor/rgb/camera_info</cameraInfoTopicName>
+        <depthImageTopicName>/xtion_sensor/depth/image_raw</depthImageTopicName>
+        <depthImageCameraInfoTopicName>/xtion_sensor/depth/camera_info</depthImageCameraInfoTopicName>
+        <pointCloudTopicName>/xtion_sensor/depth/points</pointCloudTopicName>
+        <frameName>link_xtion_optical</frameName>
         <pointCloudCutoff>0.35</pointCloudCutoff>
         <distortionK1>0.00000001</distortionK1>
@@ -108,4 +114,4 @@
       </plugin>
     </sensor>
-  </gazebo> -->
+  </gazebo>
 </robot>

File: panda_description/urdf/panda_arm.xacro (robot description, xacro)
@@ -3,20 +3,13 @@
   <xacro:macro name="panda_arm" params="name:='arm' xyz:='0 0 0' rpy:='0 0 0'">
     <link name="link_${name}_base" />
-<!--       <visual>
-        <origin xyz="${xyz}" rpy="${rpy}" />
-        <geometry>
-          <box size="0.05 0.05 0.05" />
-        </geometry>
-      </visual>
-    </link> -->
     <link name="link_${name}_0">
       <visual>
         <geometry>
-          <mesh filename="package://panda_description/meshes/visual/link0.dae" />
-        </geometry>
-      </visual>
-      <collision>
-        <geometry>
-          <mesh filename="package://panda_description/meshes/collision/link0.stl" />
+          <mesh filename="package://panda_description/meshes/visual/link_${name}_0.dae" />
+        </geometry>
+      </visual>
+      <collision>
+        <geometry>
+          <mesh filename="package://panda_description/meshes/collision/link_${name}_0.stl" />
         </geometry>
       </collision>
@@ -30,5 +23,5 @@
       </inertial>
     </link>
-    <joint name="$joint_${name}_base" type="fixed">
+    <joint name="joint_${name}_base" type="fixed">
       <origin xyz="${xyz}" rpy="${rpy}" />
       <parent link="link_${name}_base" />
@@ -38,10 +31,10 @@
       <visual>
         <geometry>
-          <mesh filename="package://panda_description/meshes/visual/link1.dae" />
-        </geometry>
-      </visual>
-      <collision>
-        <geometry>
-          <mesh filename="package://panda_description/meshes/collision/link1.stl" />
+          <mesh filename="package://panda_description/meshes/visual/link_${name}_1.dae" />
+        </geometry>
+      </visual>
+      <collision>
+        <geometry>
+          <mesh filename="package://panda_description/meshes/collision/link_${name}_1.stl" />
         </geometry>
       </collision>
@@ -66,10 +59,10 @@
       <visual>
         <geometry>
-          <mesh filename="package://panda_description/meshes/visual/link2.dae" />
-        </geometry>
-      </visual>
-      <collision>
-        <geometry>
-          <mesh filename="package://panda_description/meshes/collision/link2.stl" />
+          <mesh filename="package://panda_description/meshes/visual/link_${name}_2.dae" />
+        </geometry>
+      </visual>
+      <collision>
+        <geometry>
+          <mesh filename="package://panda_description/meshes/collision/link_${name}_2.stl" />
         </geometry>
       </collision>
@@ -94,10 +87,10 @@
       <visual>
         <geometry>
-          <mesh filename="package://panda_description/meshes/visual/link3.dae"/>
-        </geometry>
-      </visual>
-      <collision>
-        <geometry>
-          <mesh filename="package://panda_description/meshes/collision/link3.stl" />
+          <mesh filename="package://panda_description/meshes/visual/link_${name}_3.dae"/>
+        </geometry>
+      </visual>
+      <collision>
+        <geometry>
+          <mesh filename="package://panda_description/meshes/collision/link_${name}_3.stl" />
         </geometry>
       </collision>
@@ -122,10 +115,10 @@
       <visual>
         <geometry>
-          <mesh filename="package://panda_description/meshes/visual/link4.dae" />
-        </geometry>
-      </visual>
-      <collision>
-        <geometry>
-          <mesh filename="package://panda_description/meshes/collision/link4.stl" />
+          <mesh filename="package://panda_description/meshes/visual/link_${name}_4.dae" />
+        </geometry>
+      </visual>
+      <collision>
+        <geometry>
+          <mesh filename="package://panda_description/meshes/collision/link_${name}_4.stl" />
         </geometry>
       </collision>
@@ -151,10 +144,10 @@
       <visual>
         <geometry>
-          <mesh filename="package://panda_description/meshes/visual/link5.dae" />
-        </geometry>
-      </visual>
-      <collision>
-        <geometry>
-          <mesh filename="package://panda_description/meshes/collision/link5.stl" />
+          <mesh filename="package://panda_description/meshes/visual/link_${name}_5.dae" />
+        </geometry>
+      </visual>
+      <collision>
+        <geometry>
+          <mesh filename="package://panda_description/meshes/collision/link_${name}_5.stl" />
         </geometry>
       </collision>
@@ -179,10 +172,10 @@
       <visual>
         <geometry>
-          <mesh filename="package://panda_description/meshes/visual/link6.dae" />
-        </geometry>
-      </visual>
-      <collision>
-        <geometry>
-          <mesh filename="package://panda_description/meshes/collision/link6.stl" />
+          <mesh filename="package://panda_description/meshes/visual/link_${name}_6.dae" />
+        </geometry>
+      </visual>
+      <collision>
+        <geometry>
+          <mesh filename="package://panda_description/meshes/collision/link_${name}_6.stl" />
         </geometry>
       </collision>
@@ -207,10 +200,10 @@
       <visual>
         <geometry>
-          <mesh filename="package://panda_description/meshes/visual/link7.dae" />
-        </geometry>
-      </visual>
-      <collision>
-        <geometry>
-          <mesh filename="package://panda_description/meshes/collision/link7.stl" />
+          <mesh filename="package://panda_description/meshes/visual/link_${name}_7.dae" />
+        </geometry>
+      </visual>
+      <collision>
+        <geometry>
+          <mesh filename="package://panda_description/meshes/collision/link_${name}_7.stl" />
         </geometry>
       </collision>

File: panda_description/urdf/panda_arm_hand.urdf.xacro (robot description, xacro)
@@ -1,7 +1,13 @@
 <?xml version="1.0" encoding="utf-8"?>
 <robot name="panda" xmlns:xacro="http://www.ros.org/wiki/xacro">
+  <xacro:property name="deg_to_rad" value="0.01745329251994329577"/>
   <xacro:include filename="$(find panda_description)/urdf/panda_arm.xacro" />
   <xacro:include filename="$(find panda_description)/urdf/panda_hand.xacro" />
+  <xacro:include filename="$(find panda_description)/urdf/panda_xtion.xacro" />
   <xacro:panda_arm />
-  <xacro:panda_hand rpy="0 0 ${-pi/4}" />
+  <xacro:panda_hand />
+  <xacro:panda_xtion >
+    <origin xyz="0.2 0 1.4" rpy="0 ${45.0 * deg_to_rad} 0" />
+    <origin xyz="0 0 0" rpy="${-90.0 * deg_to_rad} 0 ${-90.0 * deg_to_rad}" />
+  </xacro:panda_xtion>
 </robot>

File: panda_description/urdf/panda_hand.xacro (robot description, xacro)
@@ -1,14 +1,14 @@
 <?xml version="1.0" encoding="utf-8"?>
 <robot name="panda_hand" xmlns:xacro="http://www.ros.org/wiki/xacro">
-  <xacro:macro name="panda_hand" params="name:='hand' parent:='link_arm_8'  rpy:='0 0 0' xyz:='0 0 0'">
+  <xacro:macro name="panda_hand" params="name:='hand' parent:='arm_8' rpy:='0 0 0' xyz:='0 0 0'">
     <link name="link_${name}">
       <visual>
         <geometry>
-          <mesh filename="package://panda_description/meshes/visual/hand.dae" />
+          <mesh filename="package://panda_description/meshes/visual/link_${name}.dae" />
         </geometry>
       </visual>
       <collision>
         <geometry>
-          <mesh filename="package://panda_description/meshes/collision/hand.stl" />
+          <mesh filename="package://panda_description/meshes/collision/link_${name}.stl" />
         </geometry>
       </collision>
@@ -23,6 +23,6 @@
     </link>
     <joint name="joint_${name}" type="fixed">
-      <origin xyz="${xyz}" rpy="${rpy}" />
-      <parent link="${parent}" />
+      <origin xyz="${xyz}" rpy="0 0 ${-pi/4}" />
+      <parent link="link_${parent}" />
       <child link="link_${name}" />
     </joint>
@@ -30,10 +30,10 @@
       <visual>
         <geometry>
-          <mesh filename="package://panda_description/meshes/visual/finger.dae" />
+          <mesh filename="package://panda_description/meshes/visual/link_finger.dae" />
         </geometry>
       </visual>
       <collision>
         <geometry>
-          <mesh filename="package://panda_description/meshes/collision/finger.stl" />
+          <mesh filename="package://panda_description/meshes/collision/link_finger.stl" />
         </geometry>
       </collision>
@@ -51,5 +51,5 @@
         <origin xyz="0 0 0" rpy="0 0 ${pi}" />
         <geometry>
-          <mesh filename="package://panda_description/meshes/visual/finger.dae" />
+          <mesh filename="package://panda_description/meshes/visual/link_finger.dae" />
         </geometry>
       </visual>
@@ -57,5 +57,5 @@
         <origin xyz="0 0 0" rpy="0 0 ${pi}" />
         <geometry>
-          <mesh filename="package://panda_description/meshes/collision/finger.stl" />
+          <mesh filename="package://panda_description/meshes/collision/link_finger.stl" />
         </geometry>
       </collision>
